File: Bridge_Ethernet/DriversSerie0.sch (KiCad schematic (older format))
At the start: 12 parts, among them U11 MAX3222CDW, U12 ISL83485

Commit message: Esquemático Finalizado, sin warnings. Haciendo asignaciones de footprints
Parts:
- U11: footprint SOIC127P1032X265-20N -> MAX3222CDW:SOIC127P1032X265-20N
- U12: footprint (none) -> SOIC127P600X175-8N:SOIC127P600X175-8N
Changed lines of the file:
@@
 AR Path="/5DA10068/5D8B9205" Ref="U?"  Part="1"
 AR Path="/5DA10434/5D8B9205" Ref="U?"  Part="1"
+AR Path="/5D8B9205" Ref="U11"  Part="1"
 F 0 "U11" H 4200 4170 50  0000 C CNN
 F 1 "MAX3222CDW" H 4200 4079 50  0000 C CNN
-F 2 "SOIC127P1032X265-20N" H 4200 2800 50  0001 L BNN
+F 2 "MAX3222CDW:SOIC127P1032X265-20N" H 4200 2800 50  0001 L BNN
 F 3 "Unavailable" H 4200 2800 50  0001 L BNN
 F 4 "3-V to 5.5-V Multichannel S-232 Line Driver/ eceiver 20-SOIC 0 to 70" H 4200 2800 50  0001 L BNN "Field4"
@@
 F 0 "U12" H 5900 5850 50  0000 C CNN
 F 1 "ISL83485" H 6000 5750 50  0000 C CNN
-F 2 "" H 5900 6650 50  0001 C CNN
+F 2 "SOIC127P600X175-8N:SOIC127P600X175-8N" H 5900 6650 50  0001 C CNN
 F 3 "" H 5900 6650 50  0001 C CNN
 	1    5200 5750

Commit message: Esquemático Finalizado. Asignaciones Realizadas. Comienzo de PCB.
Parts:
- C24, C25, C26, C27, C28, C29: footprint (none) -> Capacitor_SMD:C_0805_2012Metric
- D10, D9: footprint (none) -> Diode_SMD:D_SMB_Modified
- R10, R11: footprint (none) -> Resistor_SMD:R_0805_2012Metric
Changed lines of the file:
@@
 F 0 "C26" H 3115 1346 50  0000 L CNN
 F 1 "0.1uF" H 3115 1255 50  0000 L CNN
-F 2 "" H 3038 1150 50  0001 C CNN
+F 2 "Capacitor_SMD:C_0805_2012Metric" H 3038 1150 50  0001 C CNN
 F 3 "~" H 3000 1300 50  0001 C CNN
 	1    3000 1300
@@
 F 0 "C27" V 3150 2900 50  0000 C CNN
 F 1 "0.1uF" V 3150 3150 50  0000 C CNN
-F 2 "" H 3238 2850 50  0001 C CNN
+F 2 "Capacitor_SMD:C_0805_2012Metric" H 3238 2850 50  0001 C CNN
 F 3 "~" H 3200 3000 50  0001 C CNN
 	1    3200 3000
@@
 F 0 "C28" V 3150 3300 50  0000 C CNN
 F 1 "0.1uF" V 3150 3550 50  0000 C CNN
-F 2 "" H 3238 3250 50  0001 C CNN
+F 2 "Capacitor_SMD:C_0805_2012Metric" H 3238 3250 50  0001 C CNN
 F 3 "~" H 3200 3400 50  0001 C CNN
 	1    3200 3400
@@
 F 0 "C24" V 2550 2800 50  0000 C CNN
 F 1 "0.1uF" V 2550 3050 50  0000 C CNN
-F 2 "" H 2638 2750 50  0001 C CNN
+F 2 "Capacitor_SMD:C_0805_2012Metric" H 2638 2750 50  0001 C CNN
 F 3 "~" H 2600 2900 50  0001 C CNN
 	1    2600 2900
@@
 F 0 "C25" V 2550 3400 50  0000 C CNN
 F 1 "0.1uF" V 2550 3650 50  0000 C CNN
-F 2 "" H 2638 3350 50  0001 C CNN
+F 2 "Capacitor_SMD:C_0805_2012Metric" H 2638 3350 50  0001 C CNN
 F 3 "~" H 2600 3500 50  0001 C CNN
 	1    2600 3500
@@
 F 0 "C29" H 5965 4346 50  0000 L CNN
 F 1 "0.1uF" H 5965 4255 50  0000 L CNN
-F 2 "" H 5888 4150 50  0001 C CNN
+F 2 "Capacitor_SMD:C_0805_2012Metric" H 5888 4150 50  0001 C CNN
 F 3 "~" H 5850 4300 50  0001 C CNN
 	1    5850 4300
@@
 F 0 "R10" H 6620 4946 50  0000 L CNN
 F 1 "4K7" H 6620 4855 50  0000 L CNN
-F 2 "" V 6480 4900 50  0001 C CNN
+F 2 "Resistor_SMD:R_0805_2012Metric" V 6480 4900 50  0001 C CNN
 F 3 "~" H 6550 4900 50  0001 C CNN
 	1    6550 4900
@@
 F 0 "R11" H 6620 5746 50  0000 L CNN
 F 1 "4K7" H 6620 5655 50  0000 L CNN
-F 2 "" V 6480 5700 50  0001 C CNN
+F 2 "Resistor_SMD:R_0805_2012Metric" V 6480 5700 50  0001 C CNN
 F 3 "~" H 6550 5700 50  0001 C CNN
 	1    6550 5700
@@
 F 0 "D9" H 8325 2575 50  0000 C CNN
 F 1 "GL05T-E3-08" H 8325 2484 50  0000 C CNN
-F 2 "" H 8450 2100 50  0001 C CNN
+F 2 "Diode_SMD:D_SMB_Modified" H 8450 2100 50  0001 C CNN
 F 3 "" H 8450 2100 50  0001 C CNN
 	1    8400 2050
@@
 F 0 "D10" H 8325 3725 50  0000 C CNN
 F 1 "GL05T-E3-08" H 8325 3634 50  0000 C CNN
-F 2 "" H 8450 3250 50  0001 C CNN
+F 2 "Diode_SMD:D_SMB_Modified" H 8450 3250 50  0001 C CNN
 F 3 "" H 8450 3250 50  0001 C CNN
 	1    8400 3200

Commit message: Esquemático Finalizado. Asignaciones Realizadas. Componentes acomodados en PCB.
Parts:
- D10: symbol Bridge_Ethernet-rescue:GL05T-E3-08-GL05T-E3-08 -> GL05T-E3-08:GL05T-E3-08
- renumbered C24 to C26, C25 to C27, C26 to C28, C27 to C29, C28 to C30, C29 to C31, R11 to R10, R10 to R9, U11 to U10, U12 to U11
Connections:
- net B_485_0: now also D10.1; no longer D10.IN (1)
- net GND: now also D10.2, D9.2
- removed net GNDREF: D10.GND (2), D9.2
Other:
- moved on the sheet: D10

Commit message: Esquemático Finalizado. Asignaciones Realizadas. Reacomodamiento de componentes. Inicio de Ruteo.
Parts:
- D10, D9: footprint Diode_SMD:D_SMB_Modified -> SOT95P280X125-3N:SOT95P280X125-3N
Changed lines of the file:
@@
 F 0 "D9" H 8325 2575 50  0000 C CNN
 F 1 "GL05T-E3-08" H 8325 2484 50  0000 C CNN
-F 2 "Diode_SMD:D_SMB_Modified" H 8450 2100 50  0001 C CNN
+F 2 "SOT95P280X125-3N:SOT95P280X125-3N" H 8450 2100 50  0001 C CNN
 F 3 "" H 8450 2100 50  0001 C CNN
 	1    8400 2050
@@
 F 0 "D10" H 8325 3725 50  0000 C CNN
 F 1 "GL05T-E3-08" H 8325 3634 50  0000 C CNN
-F 2 "Diode_SMD:D_SMB_Modified" H 8450 3250 50  0001 C CNN
+F 2 "SOT95P280X125-3N:SOT95P280X125-3N" H 8450 3250 50  0001 C CNN
 F 3 "" H 8450 3250 50  0001 C CNN
 	1    8400 3200
