File: Bridge_Ethernet/DriversSerie1.sch (KiCad schematic (older format))
At the start: 12 parts, among them U1 MAX3222CDW, U2 ISL83485

Commit message: Esquemático Finalizado, sin warnings. Haciendo asignaciones de footprints
Parts:
- U1: footprint SOIC127P1032X265-20N -> MAX3222CDW:SOIC127P1032X265-20N
- U2: footprint (none) -> SOIC127P600X175-8N:SOIC127P600X175-8N
Changed lines of the file:
@@
 AR Path="/5DA1006A/5DE5D79D" Ref="U?"  Part="1"
 AR Path="/5DA10436/5DE5D79D" Ref="U?"  Part="1"
+AR Path="/5DE5D79D" Ref="U1"  Part="1"
 F 0 "U1" H 4200 4170 50  0000 C CNN
 F 1 "MAX3222CDW" H 4200 4079 50  0000 C CNN
-F 2 "SOIC127P1032X265-20N" H 4200 2800 50  0001 L BNN
+F 2 "MAX3222CDW:SOIC127P1032X265-20N" H 4200 2800 50  0001 L BNN
 F 3 "Unavailable" H 4200 2800 50  0001 L BNN
 F 4 "3-V to 5.5-V Multichannel S-232 Line Driver/ eceiver 20-SOIC 0 to 70" H 4200 2800 50  0001 L BNN "Field4"
@@
 F 0 "U2" H 5900 6650 50  0000 C CNN
 F 1 "ISL83485" H 5900 6550 50  0000 C CNN
-F 2 "" H 5900 6650 50  0001 C CNN
+F 2 "SOIC127P600X175-8N:SOIC127P600X175-8N" H 5900 6650 50  0001 C CNN
 F 3 "" H 5900 6650 50  0001 C CNN
 	1    5200 5750

Commit message: Esquemático Finalizado. Asignaciones Realizadas. Comienzo de PCB.
Parts:
- C1, C2, C3, C4, C5, C6: footprint (none) -> Capacitor_SMD:C_0805_2012Metric
- D4, D5: footprint (none) -> Diode_SMD:D_SMB_Modified
- R1, R2: footprint (none) -> Resistor_SMD:R_0805_2012Metric
Changed lines of the file:
@@
 F 0 "C3" H 3115 1346 50  0000 L CNN
 F 1 "0.1uF" H 3115 1255 50  0000 L CNN
-F 2 "" H 3038 1150 50  0001 C CNN
+F 2 "Capacitor_SMD:C_0805_2012Metric" H 3038 1150 50  0001 C CNN
 F 3 "~" H 3000 1300 50  0001 C CNN
 	1    3000 1300
@@
 F 0 "C4" V 3250 3150 50  0000 C CNN
 F 1 "0.1uF" V 3150 3150 50  0000 C CNN
-F 2 "" H 3238 2850 50  0001 C CNN
+F 2 "Capacitor_SMD:C_0805_2012Metric" H 3238 2850 50  0001 C CNN
 F 3 "~" H 3200 3000 50  0001 C CNN
 	1    3200 3000
@@
 F 0 "C5" V 3150 3550 50  0000 C CNN
 F 1 "0.1uF" V 3050 3550 50  0000 C CNN
-F 2 "" H 3238 3250 50  0001 C CNN
+F 2 "Capacitor_SMD:C_0805_2012Metric" H 3238 3250 50  0001 C CNN
 F 3 "~" H 3200 3400 50  0001 C CNN
 	1    3200 3400
@@
 F 0 "C6" H 5965 4346 50  0000 L CNN
 F 1 "0.1uF" H 5965 4255 50  0000 L CNN
-F 2 "" H 5888 4150 50  0001 C CNN
+F 2 "Capacitor_SMD:C_0805_2012Metric" H 5888 4150 50  0001 C CNN
 F 3 "~" H 5850 4300 50  0001 C CNN
 	1    5850 4300
@@
 F 0 "R1" H 6620 4946 50  0000 L CNN
 F 1 "4K7" H 6620 4855 50  0000 L CNN
-F 2 "" V 6480 4900 50  0001 C CNN
+F 2 "Resistor_SMD:R_0805_2012Metric" V 6480 4900 50  0001 C CNN
 F 3 "~" H 6550 4900 50  0001 C CNN
 	1    6550 4900
@@
 F 0 "R2" H 6620 5746 50  0000 L CNN
 F 1 "4K7" H 6620 5655 50  0000 L CNN
-F 2 "" V 6480 5700 50  0001 C CNN
+F 2 "Resistor_SMD:R_0805_2012Metric" V 6480 5700 50  0001 C CNN
 F 3 "~" H 6550 5700 50  0001 C CNN
 	1    6550 5700
@@
 F 0 "C2" V 2650 3650 50  0000 C CNN
 F 1 "0.1uF" V 2550 3650 50  0000 C CNN
-F 2 "" H 2638 3350 50  0001 C CNN
+F 2 "Capacitor_SMD:C_0805_2012Metric" H 2638 3350 50  0001 C CNN
 F 3 "~" H 2600 3500 50  0001 C CNN
 	1    2600 3500
@@
 F 0 "C1" V 2650 3050 50  0000 C CNN
 F 1 "0.1uF" V 2550 3050 50  0000 C CNN
-F 2 "" H 2638 2750 50  0001 C CNN
+F 2 "Capacitor_SMD:C_0805_2012Metric" H 2638 2750 50  0001 C CNN
 F 3 "~" H 2600 2900 50  0001 C CNN
 	1    2600 2900
@@
 F 0 "D4" H 8525 2675 50  0000 C CNN
 F 1 "GL05T-E3-08" H 8525 2584 50  0000 C CNN
-F 2 "" H 8650 2200 50  0001 C CNN
+F 2 "Diode_SMD:D_SMB_Modified" H 8650 2200 50  0001 C CNN
 F 3 "" H 8650 2200 50  0001 C CNN
 	1    8600 2150
@@
 F 0 "D5" H 8525 3825 50  0000 C CNN
 F 1 "GL05T-E3-08" H 8525 3734 50  0000 C CNN
-F 2 "" H 8650 3350 50  0001 C CNN
+F 2 "Diode_SMD:D_SMB_Modified" H 8650 3350 50  0001 C CNN
 F 3 "" H 8650 3350 50  0001 C CNN
 	1    8600 3300

Commit message: Esquemático Finalizado. Asignaciones Realizadas. Componentes acomodados en PCB.
Parts:
- renumbered D4 to D1, D5 to D2
Connections:
- net GNDREF is gone; now on net GND: D1.2, D2.2
Changed lines of the file:
@@
 AR Path="/5DA1006A/5DE5D79D" Ref="U?"  Part="1"
 AR Path="/5DA10436/5DE5D79D" Ref="U?"  Part="1"
-AR Path="/5DE5D79D" Ref="U1"  Part="1"
+AR Path="/5DE5D79D" Ref="U?"  Part="1"
 F 0 "U1" H 4200 4170 50  0000 C CNN
 F 1 "MAX3222CDW" H 4200 4079 50  0000 C CNN
@@
 $EndComp
 $Comp
-L power:GND #PWR05
+L power:GND #PWR03
 U 1 1 5DE5D7A6
 P 3000 1550
-AR Path="/5DA0E587/5DE5D7A6" Ref="#PWR05"  Part="1"
+AR Path="/5DA0E587/5DE5D7A6" Ref="#PWR03"  Part="1"
 AR Path="/5DA1006A/5DE5D7A6" Ref="#PWR?"  Part="1"
 AR Path="/5DA10436/5DE5D7A6" Ref="#PWR?"  Part="1"
-F 0 "#PWR05" H 3000 1300 50  0001 C CNN
+F 0 "#PWR03" H 3000 1300 50  0001 C CNN
 F 1 "GND" H 3150 1500 50  0000 C CNN
 F 2 "" H 3000 1550 50  0001 C CNN
@@
 	3000 1450 3000 1550
 $Comp
-L power:+3V3 #PWR04
+L power:+3V3 #PWR02
 U 1 1 5D8BB06E
 P 3000 900
-AR Path="/5DA0E587/5D8BB06E" Ref="#PWR04"  Part="1"
+AR Path="/5DA0E587/5D8BB06E" Ref="#PWR02"  Part="1"
 AR Path="/5DA1006A/5D8BB06E" Ref="#PWR?"  Part="1"
 AR Path="/5DA10436/5D8BB06E" Ref="#PWR?"  Part="1"
-F 0 "#PWR04" H 3000 750 50  0001 C CNN
+F 0 "#PWR02" H 3000 750 50  0001 C CNN
 F 1 "+3V3" H 3015 1073 50  0000 C CNN
 F 2 "" H 3000 900 50  0001 C CNN
@@
 	3000 1050 3000 1150
 $Comp
-L power:GND #PWR06
+L power:GND #PWR04
 U 1 1 5D8C18CC
 P 3400 2150
-AR Path="/5DA0E587/5D8C18CC" Ref="#PWR06"  Part="1"
+AR Path="/5DA0E587/5D8C18CC" Ref="#PWR04"  Part="1"
 AR Path="/5DA1006A/5D8C18CC" Ref="#PWR?"  Part="1"
 AR Path="/5DA10436/5D8C18CC" Ref="#PWR?"  Part="1"
-F 0 "#PWR06" H 3400 1900 50  0001 C CNN
+F 0 "#PWR04" H 3400 1900 50  0001 C CNN
 F 1 "GND" H 3250 2100 50  0000 C CNN
 F 2 "" H 3400 2150 50  0001 C CNN
@@
 NoConn ~ 4900 2200
 $Comp
-L power:GND #PWR07
+L power:GND #PWR05
 U 1 1 5DE5D7AC
 P 3500 4100
-AR Path="/5DA0E587/5DE5D7AC" Ref="#PWR07"  Part="1"
+AR Path="/5DA0E587/5DE5D7AC" Ref="#PWR05"  Part="1"
 AR Path="/5DA1006A/5DE5D7AC" Ref="#PWR?"  Part="1"
 AR Path="/5DA10436/5DE5D7AC" Ref="#PWR?"  Part="1"
-F 0 "#PWR07" H 3500 3850 50  0001 C CNN
+F 0 "#PWR05" H 3500 3850 50  0001 C CNN
 F 1 "GND" H 3350 4050 50  0000 C CNN
 F 2 "" H 3500 4100 50  0001 C CNN
@@
 	5850 4450 5850 4550
 $Comp
-L power:+3V3 #PWR09
+L power:+3V3 #PWR07
 U 1 1 5DE5D7C9
 P 5850 3900
-AR Path="/5DA0E587/5DE5D7C9" Ref="#PWR09"  Part="1"
+AR Path="/5DA0E587/5DE5D7C9" Ref="#PWR07"  Part="1"
 AR Path="/5DA1006A/5DE5D7C9" Ref="#PWR?"  Part="1"
 AR Path="/5DA10436/5DE5D7C9" Ref="#PWR?"  Part="1"
-F 0 "#PWR09" H 5850 3750 50  0001 C CNN
+F 0 "#PWR07" H 5850 3750 50  0001 C CNN
 F 1 "+3V3" H 5865 4073 50  0000 C CNN
 F 2 "" H 5850 3900 50  0001 C CNN
@@
 $EndComp
 $Comp
-L power:GND #PWR010
+L power:GND #PWR08
 U 1 1 5D8DF5E3
 P 5850 4550
-AR Path="/5DA0E587/5D8DF5E3" Ref="#PWR010"  Part="1"
+AR Path="/5DA0E587/5D8DF5E3" Ref="#PWR08"  Part="1"
 AR Path="/5DA1006A/5D8DF5E3" Ref="#PWR?"  Part="1"
 AR Path="/5DA10436/5D8DF5E3" Ref="#PWR?"  Part="1"
-F 0 "#PWR010" H 5850 4300 50  0001 C CNN
+F 0 "#PWR08" H 5850 4300 50  0001 C CNN
 F 1 "GND" H 6000 4500 50  0000 C CNN
 F 2 "" H 5850 4550 50  0001 C CNN
@@
 	5850 4100 5850 4150
 $Comp
-L power:GND #PWR08
+L power:GND #PWR06
 U 1 1 5DE5D7CA
 P 5700 6050
-AR Path="/5DA0E587/5DE5D7CA" Ref="#PWR08"  Part="1"
+AR Path="/5DA0E587/5DE5D7CA" Ref="#PWR06"  Part="1"
 AR Path="/5DA1006A/5DE5D7CA" Ref="#PWR?"  Part="1"
 AR Path="/5DA10436/5DE5D7CA" Ref="#PWR?"  Part="1"
-F 0 "#PWR08" H 5700 5800 50  0001 C CNN
+F 0 "#PWR06" H 5700 5800 50  0001 C CNN
 F 1 "GND" H 5550 6000 50  0000 C CNN
 F 2 "" H 5700 6050 50  0001 C CNN
@@
 	1300 2300 3500 2300
 $Comp
-L power:GND #PWR03
+L power:GND #PWR01
 U 1 1 5DE5D7BB
 P 2350 3700
-AR Path="/5DA0E587/5DE5D7BB" Ref="#PWR03"  Part="1"
+AR Path="/5DA0E587/5DE5D7BB" Ref="#PWR01"  Part="1"
 AR Path="/5DA1006A/5DE5D7BB" Ref="#PWR?"  Part="1"
 AR Path="/5DA10436/5DE5D7BB" Ref="#PWR?"  Part="1"
-F 0 "#PWR03" H 2350 3450 50  0001 C CNN
+F 0 "#PWR01" H 2350 3450 50  0001 C CNN
 F 1 "GND" H 2200 3650 50  0000 C CNN
 F 2 "" H 2350 3700 50  0001 C CNN
@@
 AR Path="/5D9FFB34/5DC696EA" Ref="D?"  Part="1"
 AR Path="/5DA0E4A1/5DC696EA" Ref="D?"  Part="1"
-AR Path="/5DA0E587/5DC696EA" Ref="D4"  Part="1"
-AR Path="/5DC696EA" Ref="D4"  Part="1"
-F 0 "D4" H 8525 2675 50  0000 C CNN
+AR Path="/5DA0E587/5DC696EA" Ref="D1"  Part="1"
+AR Path="/5DC696EA" Ref="D?"  Part="1"
+F 0 "D1" H 8525 2675 50  0000 C CNN
 F 1 "GL05T-E3-08" H 8525 2584 50  0000 C CNN
 F 2 "Diode_SMD:D_SMB_Modified" H 8650 2200 50  0001 C CNN
@@
 AR Path="/5D9FFB34/5DC696F0" Ref="D?"  Part="1"
 AR Path="/5DA0E4A1/5DC696F0" Ref="D?"  Part="1"
-AR Path="/5DA0E587/5DC696F0" Ref="D5"  Part="1"
-AR Path="/5DC696F0" Ref="D5"  Part="1"
-F 0 "D5" H 8525 3825 50  0000 C CNN
+AR Path="/5DA0E587/5DC696F0" Ref="D2"  Part="1"
+AR Path="/5DC696F0" Ref="D?"  Part="1"
+F 0 "D2" H 8525 3825 50  0000 C CNN
 F 1 "GL05T-E3-08" H 8525 3734 50  0000 C CNN
 F 2 "Diode_SMD:D_SMB_Modified" H 8650 3350 50  0001 C CNN
@@
 	1    0    0    -1
 $EndComp
-$Comp
-L power:GNDREF #PWR?
-U 1 1 5DC696F6
-P 8350 2150
-AR Path="/5D9FFB34/5DC696F6" Ref="#PWR?"  Part="1"
-AR Path="/5DA0E4A1/5DC696F6" Ref="#PWR?"  Part="1"
-AR Path="/5DA0E587/5DC696F6" Ref="#PWR01"  Part="1"
-F 0 "#PWR01" H 8350 1900 50  0001 C CNN
-F 1 "GNDREF" H 8355 1977 50  0001 C CNN
-F 2 "" H 8350 2150 50  0001 C CNN
-F 3 "" H 8350 2150 50  0001 C CNN
-	1    8350 2150
-	1    0    0    -1
-$EndComp
 Wire Wire Line
 	8350 2150 8350 2050
-$Comp
-L power:GNDREF #PWR?
-U 1 1 5DC696FD
-P 8350 3300
-AR Path="/5D9FFB34/5DC696FD" Ref="#PWR?"  Part="1"
-AR Path="/5DA0E4A1/5DC696FD" Ref="#PWR?"  Part="1"
-AR Path="/5DA0E587/5DC696FD" Ref="#PWR02"  Part="1"
-F 0 "#PWR02" H 8350 3050 50  0001 C CNN
-F 1 "GNDREF" H 8355 3127 50  0001 C CNN
-F 2 "" H 8350 3300 50  0001 C CNN
-F 3 "" H 8350 3300 50  0001 C CNN
-	1    8350 3300
-	1    0    0    -1
-$EndComp
 Wire Wire Line
 	8350 3300 8350 3200
@@
 Text HLabel 7450 5450 2    50   Input ~ 0
 B_485_1
+$Comp
+L power:GND #PWR?
+U 1 1 5DC9A9B3
+P 8350 2150
+AR Path="/5D9FFB34/5DC9A9B3" Ref="#PWR?"  Part="1"
+AR Path="/5DA0E587/5DC9A9B3" Ref="#PWR09"  Part="1"
+F 0 "#PWR09" H 8350 1900 50  0001 C CNN
+F 1 "GND" H 8355 1977 50  0000 C CNN
+F 2 "" H 8350 2150 50  0001 C CNN
+F 3 "" H 8350 2150 50  0001 C CNN
+	1    8350 2150
+	1    0    0    -1
+$EndComp
+$Comp
+L power:GND #PWR?
+U 1 1 5DC9BC19
+P 8350 3300
+AR Path="/5D9FFB34/5DC9BC19" Ref="#PWR?"  Part="1"
+AR Path="/5DA0E587/5DC9BC19" Ref="#PWR010"  Part="1"
+F 0 "#PWR010" H 8350 3050 50  0001 C CNN
+F 1 "GND" H 8355 3127 50  0000 C CNN
+F 2 "" H 8350 3300 50  0001 C CNN
+F 3 "" H 8350 3300 50  0001 C CNN
+	1    8350 3300
+	1    0    0    -1
+$EndComp
 $EndSCHEMATC

Commit message: Esquemático Finalizado. Asignaciones Realizadas. Reacomodamiento de componentes. Inicio de Ruteo.
Parts:
- D1, D2: footprint Diode_SMD:D_SMB_Modified -> SOT95P280X125-3N:SOT95P280X125-3N
Changed lines of the file:
@@
 F 0 "D1" H 8525 2675 50  0000 C CNN
 F 1 "GL05T-E3-08" H 8525 2584 50  0000 C CNN
-F 2 "Diode_SMD:D_SMB_Modified" H 8650 2200 50  0001 C CNN
+F 2 "SOT95P280X125-3N:SOT95P280X125-3N" H 8650 2200 50  0001 C CNN
 F 3 "" H 8650 2200 50  0001 C CNN
 	1    8600 2150
@@
 F 0 "D2" H 8525 3825 50  0000 C CNN
 F 1 "GL05T-E3-08" H 8525 3734 50  0000 C CNN
-F 2 "Diode_SMD:D_SMB_Modified" H 8650 3350 50  0001 C CNN
+F 2 "SOT95P280X125-3N:SOT95P280X125-3N" H 8650 3350 50  0001 C CNN
 F 3 "" H 8650 3350 50  0001 C CNN
 	1    8600 3300
