File: Bridge_Ethernet/DriversSerie3.sch (KiCad schematic (older format))
At the start: 12 parts, among them U5 MAX3222CDW, U6 ISL83485

Commit message: Esquemático Finalizado, sin warnings. Haciendo asignaciones de footprints
Parts:
- U5: footprint SOIC127P1032X265-20N -> MAX3222CDW:SOIC127P1032X265-20N
- U6: footprint (none) -> SOIC127P600X175-8N:SOIC127P600X175-8N
Changed lines of the file:
@@
 F 0 "U5" H 4200 4170 50  0000 C CNN
 F 1 "MAX3222CDW" H 4200 4079 50  0000 C CNN
-F 2 "SOIC127P1032X265-20N" H 4200 2800 50  0001 L BNN
+F 2 "MAX3222CDW:SOIC127P1032X265-20N" H 4200 2800 50  0001 L BNN
 F 3 "Unavailable" H 4200 2800 50  0001 L BNN
 F 4 "3-V to 5.5-V Multichannel S-232 Line Driver/ eceiver 20-SOIC 0 to 70" H 4200 2800 50  0001 L BNN "Field4"
@@
 F 0 "U6" H 5900 5850 50  0000 C CNN
 F 1 "ISL83485" H 6000 5750 50  0000 C CNN
-F 2 "" H 5900 6650 50  0001 C CNN
+F 2 "SOIC127P600X175-8N:SOIC127P600X175-8N" H 5900 6650 50  0001 C CNN
 F 3 "" H 5900 6650 50  0001 C CNN
 	1    5200 5750

Commit message: Esquemático Finalizado. Asignaciones Realizadas. Comienzo de PCB.
Parts:
- C13, C14, C15, C16, C17, C18: footprint (none) -> Capacitor_SMD:C_0805_2012Metric
- D11, D12: footprint (none) -> Diode_SMD:D_SMB_Modified
- R5, R6: footprint (none) -> Resistor_SMD:R_0805_2012Metric
Changed lines of the file:
@@
 F 0 "C15" H 3115 1346 50  0000 L CNN
 F 1 "0.1uF" H 3115 1255 50  0000 L CNN
-F 2 "" H 3038 1150 50  0001 C CNN
+F 2 "Capacitor_SMD:C_0805_2012Metric" H 3038 1150 50  0001 C CNN
 F 3 "~" H 3000 1300 50  0001 C CNN
 	1    3000 1300
@@
 F 0 "C16" V 3250 3150 50  0000 C CNN
 F 1 "0.1uF" V 3150 3150 50  0000 C CNN
-F 2 "" H 3238 2850 50  0001 C CNN
+F 2 "Capacitor_SMD:C_0805_2012Metric" H 3238 2850 50  0001 C CNN
 F 3 "~" H 3200 3000 50  0001 C CNN
 	1    3200 3000
@@
 F 0 "C17" V 3150 3550 50  0000 C CNN
 F 1 "0.1uF" V 3050 3550 50  0000 C CNN
-F 2 "" H 3238 3250 50  0001 C CNN
+F 2 "Capacitor_SMD:C_0805_2012Metric" H 3238 3250 50  0001 C CNN
 F 3 "~" H 3200 3400 50  0001 C CNN
 	1    3200 3400
@@
 F 0 "C18" H 5965 4346 50  0000 L CNN
 F 1 "0.1uF" H 5965 4255 50  0000 L CNN
-F 2 "" H 5888 4150 50  0001 C CNN
+F 2 "Capacitor_SMD:C_0805_2012Metric" H 5888 4150 50  0001 C CNN
 F 3 "~" H 5850 4300 50  0001 C CNN
 	1    5850 4300
@@
 F 0 "R5" H 6620 4946 50  0000 L CNN
 F 1 "4K7" H 6620 4855 50  0000 L CNN
-F 2 "" V 6480 4900 50  0001 C CNN
+F 2 "Resistor_SMD:R_0805_2012Metric" V 6480 4900 50  0001 C CNN
 F 3 "~" H 6550 4900 50  0001 C CNN
 	1    6550 4900
@@
 F 0 "R6" H 6620 5746 50  0000 L CNN
 F 1 "4K7" H 6620 5655 50  0000 L CNN
-F 2 "" V 6480 5700 50  0001 C CNN
+F 2 "Resistor_SMD:R_0805_2012Metric" V 6480 5700 50  0001 C CNN
 F 3 "~" H 6550 5700 50  0001 C CNN
 	1    6550 5700
@@
 F 0 "C14" V 2650 3650 50  0000 C CNN
 F 1 "0.1uF" V 2550 3650 50  0000 C CNN
-F 2 "" H 2638 3350 50  0001 C CNN
+F 2 "Capacitor_SMD:C_0805_2012Metric" H 2638 3350 50  0001 C CNN
 F 3 "~" H 2600 3500 50  0001 C CNN
 	1    2600 3500
@@
 F 0 "C13" V 2650 3050 50  0000 C CNN
 F 1 "0.1uF" V 2550 3050 50  0000 C CNN
-F 2 "" H 2638 2750 50  0001 C CNN
+F 2 "Capacitor_SMD:C_0805_2012Metric" H 2638 2750 50  0001 C CNN
 F 3 "~" H 2600 2900 50  0001 C CNN
 	1    2600 2900
@@
 F 0 "D11" H 7925 2675 50  0000 C CNN
 F 1 "GL05T-E3-08" H 7925 2584 50  0000 C CNN
-F 2 "" H 8050 2200 50  0001 C CNN
+F 2 "Diode_SMD:D_SMB_Modified" H 8050 2200 50  0001 C CNN
 F 3 "" H 8050 2200 50  0001 C CNN
 	1    8000 2150
@@
 F 0 "D12" H 7925 3825 50  0000 C CNN
 F 1 "GL05T-E3-08" H 7925 3734 50  0000 C CNN
-F 2 "" H 8050 3350 50  0001 C CNN
+F 2 "Diode_SMD:D_SMB_Modified" H 8050 3350 50  0001 C CNN
 F 3 "" H 8050 3350 50  0001 C CNN
 	1    8000 3300

Commit message: Esquemático Finalizado. Asignaciones Realizadas. Componentes acomodados en PCB.
Parts:
- renumbered C13 to C32, C14 to C33, C15 to C34, C16 to C35, C17 to C36, C18 to C37, R5 to R11, R6 to R12, U5 to U12, U6 to U13
Connections:
- net GNDREF is gone; now on net GND: D11.2, D12.2
Changed lines of the file:
@@
 $EndDescr
 $Comp
-L MAX3222CDW:MAX3222CDW U5
+L MAX3222CDW:MAX3222CDW U12
 U 1 1 5DE5D79E
 P 4200 2800
-F 0 "U5" H 4200 4170 50  0000 C CNN
+F 0 "U12" H 4200 4170 50  0000 C CNN
 F 1 "MAX3222CDW" H 4200 4079 50  0000 C CNN
 F 2 "MAX3222CDW:SOIC127P1032X265-20N" H 4200 2800 50  0001 L BNN
@@
 $EndComp
 $Comp
-L Device:C C15
+L Device:C C34
 U 1 1 5DE5D7A4
 P 3000 1300
-F 0 "C15" H 3115 1346 50  0000 L CNN
+F 0 "C34" H 3115 1346 50  0000 L CNN
 F 1 "0.1uF" H 3115 1255 50  0000 L CNN
 F 2 "Capacitor_SMD:C_0805_2012Metric" H 3038 1150 50  0001 C CNN
@@
 $EndComp
 $Comp
-L power:GND #PWR025
+L power:GND #PWR061
 U 1 1 5DE5D7A8
 P 3000 1550
-F 0 "#PWR025" H 3000 1300 50  0001 C CNN
+F 0 "#PWR061" H 3000 1300 50  0001 C CNN
 F 1 "GND" H 3150 1500 50  0000 C CNN
 F 2 "" H 3000 1550 50  0001 C CNN
@@
 	3000 1450 3000 1550
 $Comp
-L power:+3V3 #PWR024
+L power:+3V3 #PWR060
 U 1 1 5DE5D7A0
 P 3000 900
-F 0 "#PWR024" H 3000 750 50  0001 C CNN
+F 0 "#PWR060" H 3000 750 50  0001 C CNN
 F 1 "+3V3" H 3015 1073 50  0000 C CNN
 F 2 "" H 3000 900 50  0001 C CNN
@@
 	3000 1050 3000 1150
 $Comp
-L power:GND #PWR026
+L power:GND #PWR062
 U 1 1 5DE5D7AA
 P 3400 2150
-F 0 "#PWR026" H 3400 1900 50  0001 C CNN
+F 0 "#PWR062" H 3400 1900 50  0001 C CNN
 F 1 "GND" H 3250 2100 50  0000 C CNN
 F 2 "" H 3400 2150 50  0001 C CNN
@@
 NoConn ~ 4900 2200
 $Comp
-L power:GND #PWR027
+L power:GND #PWR063
 U 1 1 5DE5D7AE
 P 3500 4100
-F 0 "#PWR027" H 3500 3850 50  0001 C CNN
+F 0 "#PWR063" H 3500 3850 50  0001 C CNN
 F 1 "GND" H 3350 4050 50  0000 C CNN
 F 2 "" H 3500 4100 50  0001 C CNN
@@
 	4900 2100 5000 2100
 $Comp
-L Device:C C16
+L Device:C C35
 U 1 1 5DE5D7B0
 P 3200 3000
-F 0 "C16" V 3250 3150 50  0000 C CNN
+F 0 "C35" V 3250 3150 50  0000 C CNN
 F 1 "0.1uF" V 3150 3150 50  0000 C CNN
 F 2 "Capacitor_SMD:C_0805_2012Metric" H 3238 2850 50  0001 C CNN
@@
 $EndComp
 $Comp
-L Device:C C17
+L Device:C C36
 U 1 1 5DE5D7B3
 P 3200 3400
-F 0 "C17" V 3150 3550 50  0000 C CNN
+F 0 "C36" V 3150 3550 50  0000 C CNN
 F 1 "0.1uF" V 3050 3550 50  0000 C CNN
 F 2 "Capacitor_SMD:C_0805_2012Metric" H 3238 3250 50  0001 C CNN
@@
 	4900 1900 5100 1900
 $Comp
-L Device:C C18
+L Device:C C37
 U 1 1 5DE5D7C1
 P 5850 4300
-F 0 "C18" H 5965 4346 50  0000 L CNN
+F 0 "C37" H 5965 4346 50  0000 L CNN
 F 1 "0.1uF" H 5965 4255 50  0000 L CNN
 F 2 "Capacitor_SMD:C_0805_2012Metric" H 5888 4150 50  0001 C CNN
@@
 	5850 4450 5850 4550
 $Comp
-L power:+3V3 #PWR029
+L power:+3V3 #PWR065
 U 1 1 5DE5D7C7
 P 5850 3900
-F 0 "#PWR029" H 5850 3750 50  0001 C CNN
+F 0 "#PWR065" H 5850 3750 50  0001 C CNN
 F 1 "+3V3" H 5865 4073 50  0000 C CNN
 F 2 "" H 5850 3900 50  0001 C CNN
@@
 $EndComp
 $Comp
-L ISL83485:ISL83485 U6
+L ISL83485:ISL83485 U13
 U 1 1 5DE5D7BF
 P 5200 5750
-F 0 "U6" H 5900 5850 50  0000 C CNN
+F 0 "U13" H 5900 5850 50  0000 C CNN
 F 1 "ISL83485" H 6000 5750 50  0000 C CNN
 F 2 "SOIC127P600X175-8N:SOIC127P600X175-8N" H 5900 6650 50  0001 C CNN
@@
 $EndComp
 $Comp
-L power:GND #PWR030
+L power:GND #PWR066
 U 1 1 5DE5D7C4
 P 5850 4550
-F 0 "#PWR030" H 5850 4300 50  0001 C CNN
+F 0 "#PWR066" H 5850 4300 50  0001 C CNN
 F 1 "GND" H 6000 4500 50  0000 C CNN
 F 2 "" H 5850 4550 50  0001 C CNN
@@
 	5850 4100 5850 4150
 $Comp
-L power:GND #PWR028
+L power:GND #PWR064
 U 1 1 5DE5D7CC
 P 5700 6050
-F 0 "#PWR028" H 5700 5800 50  0001 C CNN
+F 0 "#PWR064" H 5700 5800 50  0001 C CNN
 F 1 "GND" H 5550 6000 50  0000 C CNN
 F 2 "" H 5700 6050 50  0001 C CNN
@@
 	6150 5450 6550 5450
 $Comp
-L Device:R R5
+L Device:R R11
 U 1 1 5D8E72F0
 P 6550 4900
-F 0 "R5" H 6620 4946 50  0000 L CNN
+F 0 "R11" H 6620 4946 50  0000 L CNN
 F 1 "4K7" H 6620 4855 50  0000 L CNN
 F 2 "Resistor_SMD:R_0805_2012Metric" V 6480 4900 50  0001 C CNN
@@
 	6550 5200 7450 5200
 $Comp
-L Device:R R6
+L Device:R R12
 U 1 1 5D8E8660
 P 6550 5700
-F 0 "R6" H 6620 5746 50  0000 L CNN
+F 0 "R12" H 6620 5746 50  0000 L CNN
 F 1 "4K7" H 6620 5655 50  0000 L CNN
 F 2 "Resistor_SMD:R_0805_2012Metric" V 6480 5700 50  0001 C CNN
@@
 	1300 2300 3500 2300
 $Comp
-L power:GND #PWR023
+L power:GND #PWR059
 U 1 1 5D8C9B04
 P 2350 3700
-F 0 "#PWR023" H 2350 3450 50  0001 C CNN
+F 0 "#PWR059" H 2350 3450 50  0001 C CNN
 F 1 "GND" H 2200 3650 50  0000 C CNN
 F 2 "" H 2350 3700 50  0001 C CNN
@@
 $EndComp
 $Comp
-L Device:C C14
+L Device:C C33
 U 1 1 5D8C5510
 P 2600 3500
-F 0 "C14" V 2650 3650 50  0000 C CNN
+F 0 "C33" V 2650 3650 50  0000 C CNN
 F 1 "0.1uF" V 2550 3650 50  0000 C CNN
 F 2 "Capacitor_SMD:C_0805_2012Metric" H 2638 3350 50  0001 C CNN
@@
 $EndComp
 $Comp
-L Device:C C13
+L Device:C C32
 U 1 1 5DE5D7B6
 P 2600 2900
-F 0 "C13" V 2650 3050 50  0000 C CNN
+F 0 "C32" V 2650 3050 50  0000 C CNN
 F 1 "0.1uF" V 2550 3050 50  0000 C CNN
 F 2 "Capacitor_SMD:C_0805_2012Metric" H 2638 2750 50  0001 C CNN
@@
 AR Path="/5DA0E587/5DC9C611" Ref="D?"  Part="1"
 AR Path="/5DA1006A/5DC9C611" Ref="D11"  Part="1"
-AR Path="/5DC9C611" Ref="D11"  Part="1"
+AR Path="/5DC9C611" Ref="D?"  Part="1"
 F 0 "D11" H 7925 2675 50  0000 C CNN
 F 1 "GL05T-E3-08" H 7925 2584 50  0000 C CNN
@@
 AR Path="/5DA0E587/5DC9C617" Ref="D?"  Part="1"
 AR Path="/5DA1006A/5DC9C617" Ref="D12"  Part="1"
-AR Path="/5DC9C617" Ref="D12"  Part="1"
+AR Path="/5DC9C617" Ref="D?"  Part="1"
 F 0 "D12" H 7925 3825 50  0000 C CNN
 F 1 "GL05T-E3-08" H 7925 3734 50  0000 C CNN
@@
 	1    0    0    -1
 $EndComp
-$Comp
-L power:GNDREF #PWR?
-U 1 1 5DC9C61D
-P 7750 2150
-AR Path="/5D9FFB34/5DC9C61D" Ref="#PWR?"  Part="1"
-AR Path="/5DA0E4A1/5DC9C61D" Ref="#PWR?"  Part="1"
-AR Path="/5DA0E587/5DC9C61D" Ref="#PWR?"  Part="1"
-AR Path="/5DA1006A/5DC9C61D" Ref="#PWR031"  Part="1"
-F 0 "#PWR031" H 7750 1900 50  0001 C CNN
-F 1 "GNDREF" H 7755 1977 50  0001 C CNN
-F 2 "" H 7750 2150 50  0001 C CNN
-F 3 "" H 7750 2150 50  0001 C CNN
-	1    7750 2150
-	1    0    0    -1
-$EndComp
 Wire Wire Line
 	7750 2150 7750 2050
-$Comp
-L power:GNDREF #PWR?
-U 1 1 5DC9C624
-P 7750 3300
-AR Path="/5D9FFB34/5DC9C624" Ref="#PWR?"  Part="1"
-AR Path="/5DA0E4A1/5DC9C624" Ref="#PWR?"  Part="1"
-AR Path="/5DA0E587/5DC9C624" Ref="#PWR?"  Part="1"
-AR Path="/5DA1006A/5DC9C624" Ref="#PWR032"  Part="1"
-F 0 "#PWR032" H 7750 3050 50  0001 C CNN
-F 1 "GNDREF" H 7755 3127 50  0001 C CNN
-F 2 "" H 7750 3300 50  0001 C CNN
-F 3 "" H 7750 3300 50  0001 C CNN
-	1    7750 3300
-	1    0    0    -1
-$EndComp
 Wire Wire Line
 	7750 3300 7750 3200
@@
 Text HLabel 7550 3000 0    50   Input ~ 0
 RX_232_3
+$Comp
+L power:GND #PWR?
+U 1 1 5DCA3665
+P 7750 3300
+AR Path="/5D9FFB34/5DCA3665" Ref="#PWR?"  Part="1"
+AR Path="/5DA1006A/5DCA3665" Ref="#PWR068"  Part="1"
+F 0 "#PWR068" H 7750 3050 50  0001 C CNN
+F 1 "GND" H 7755 3127 50  0000 C CNN
+F 2 "" H 7750 3300 50  0001 C CNN
+F 3 "" H 7750 3300 50  0001 C CNN
+	1    7750 3300
+	1    0    0    -1
+$EndComp
+$Comp
+L power:GND #PWR?
+U 1 1 5DCA4D00
+P 7750 2150
+AR Path="/5D9FFB34/5DCA4D00" Ref="#PWR?"  Part="1"
+AR Path="/5DA1006A/5DCA4D00" Ref="#PWR067"  Part="1"
+F 0 "#PWR067" H 7750 1900 50  0001 C CNN
+F 1 "GND" H 7755 1977 50  0000 C CNN
+F 2 "" H 7750 2150 50  0001 C CNN
+F 3 "" H 7750 2150 50  0001 C CNN
+	1    7750 2150
+	1    0    0    -1
+$EndComp
 $EndSCHEMATC

Commit message: Esquemático Finalizado. Asignaciones Realizadas. Reacomodamiento de componentes. Inicio de Ruteo.
Parts:
- D11, D12: footprint Diode_SMD:D_SMB_Modified -> SOT95P280X125-3N:SOT95P280X125-3N
Changed lines of the file:
@@
 F 0 "D11" H 7925 2675 50  0000 C CNN
 F 1 "GL05T-E3-08" H 7925 2584 50  0000 C CNN
-F 2 "Diode_SMD:D_SMB_Modified" H 8050 2200 50  0001 C CNN
+F 2 "SOT95P280X125-3N:SOT95P280X125-3N" H 8050 2200 50  0001 C CNN
 F 3 "" H 8050 2200 50  0001 C CNN
 	1    8000 2150
@@
 F 0 "D12" H 7925 3825 50  0000 C CNN
 F 1 "GL05T-E3-08" H 7925 3734 50  0000 C CNN
-F 2 "Diode_SMD:D_SMB_Modified" H 8050 3350 50  0001 C CNN
+F 2 "SOT95P280X125-3N:SOT95P280X125-3N" H 8050 3350 50  0001 C CNN
 F 3 "" H 8050 3350 50  0001 C CNN
 	1    8000 3300
