File: Bridge_Ethernet/Fuente.sch (KiCad schematic (older format))
At the start: 14 parts, among them J3 Conn_01x04_Male, J4 Conn_01x04_Male, U10 REG1117, U9 LM2574M-5

Commit message: Esquemático Finalizado, sin warnings. Haciendo asignaciones de footprints
Parts:
- U10: footprint (none) -> REG1117:DD-3
Connections:
- net GNDREF: no longer C21.2, C22.2, C23.2, D2.3 (+), D3.2 (A), D8.2 (A), J3.1 (Pin_1), J3.2 (Pin_2), J3.3 (Pin_3), J3.4 (Pin_4), J4.1 (Pin_1), J4.2 (Pin_2), U10.1 (GND), U9.4 (SGND), U9.5 (~ON~/OFF), U9.6 (PGND)
- new net GND: C21.2, C22.2, C23.2, D2.3 (+), D3.2 (A), D8.2 (A), J3.1 (Pin_1), J3.2 (Pin_2), J3.3 (Pin_3), J3.4 (Pin_4), J4.1 (Pin_1), J4.2 (Pin_2), U10.1 (GND), U9.4 (SGND), U9.5 (~ON~/OFF), U9.6 (PGND)
Other:
- moved on the sheet: C23
Changed lines of the file:
@@
 U 1 1 5D8B1D75
 P 8750 3000
+AR Path="/5D8B1D75" Ref="U10"  Part="1"
+AR Path="/5D9FFB34/5D8B1D75" Ref="U10"  Part="1"
 F 0 "U10" H 8750 3370 50  0000 C CNN
 F 1 "REG1117" H 8750 3279 50  0000 C CNN
-F 2 "" H 8750 3000 50  0001 C CNN
+F 2 "REG1117:DD-3" H 8750 3000 50  0001 C CNN
 F 3 "Unavailable" H 8750 3000 50  0001 L BNN
 F 4 "None" H 8750 3000 50  0001 L BNN "Field4"
@@
 L Device:C C23
 U 1 1 5D8B2AEE
-P 9350 3500
-F 0 "C23" H 9465 3546 50  0000 L CNN
-F 1 "10uF" H 9465 3455 50  0000 L CNN
-F 2 "" H 9388 3350 50  0001 C CNN
-F 3 "~" H 9350 3500 50  0001 C CNN
-	1    9350 3500
+P 9600 3500
+F 0 "C23" H 9715 3546 50  0000 L CNN
+F 1 "10uF" H 9715 3455 50  0000 L CNN
+F 2 "" H 9638 3350 50  0001 C CNN
+F 3 "~" H 9600 3500 50  0001 C CNN
+	1    9600 3500
 	1    0    0    -1
 $EndComp
@@
 	7550 3350 7550 3450
 Wire Wire Line
-	6750 3000 7550 3000
-Wire Wire Line
-	9350 3000 9250 3000
+	6750 3000 7200 3000
 Connection ~ 7550 3350
 Connection ~ 7550 3000
@@
 L power:+3.3V #PWR058
 U 1 1 5D8D85F9
-P 9350 2950
-F 0 "#PWR058" H 9350 2800 50  0001 C CNN
-F 1 "+3.3V" H 9365 3123 50  0000 C CNN
-F 2 "" H 9350 2950 50  0001 C CNN
-F 3 "" H 9350 2950 50  0001 C CNN
-	1    9350 2950
-	1    0    0    -1
-$EndComp
-Wire Wire Line
-	9350 3000 9350 2950
-Connection ~ 9350 3000
+P 9600 2950
+F 0 "#PWR058" H 9600 2800 50  0001 C CNN
+F 1 "+3.3V" H 9615 3123 50  0000 C CNN
+F 2 "" H 9600 2950 50  0001 C CNN
+F 3 "" H 9600 2950 50  0001 C CNN
+	1    9600 2950
+	1    0    0    -1
+$EndComp
+Wire Wire Line
+	9300 3000 9300 2950
 $Comp
 L power:+5V #PWR054
@@
 	0    1    1    0
 $EndComp
-Wire Wire Line
-	4600 3000 5250 3000
 $Comp
 L power:GNDREF #PWR046
@@
 Wire Wire Line
 	7550 3000 8250 3000
-$Comp
-L power:GNDREF #PWR044
-U 1 1 5D95DC79
-P 1700 3900
-F 0 "#PWR044" H 1700 3650 50  0001 C CNN
-F 1 "GNDREF" H 1705 3727 50  0001 C CNN
-F 2 "" H 1700 3900 50  0001 C CNN
-F 3 "" H 1700 3900 50  0001 C CNN
-	1    1700 3900
-	1    0    0    -1
-$EndComp
 Wire Wire Line
 	1300 4150 1350 4150
@@
 Wire Wire Line
 	1700 3850 1700 3900
-Wire Wire Line
-	1300 3850 1700 3850
 Wire Wire Line
 	1300 3850 1300 3950
@@
 Connection ~ 1300 2900
 Wire Wire Line
-	1300 2900 1700 2900
-Wire Wire Line
 	1700 2900 1700 2950
-$Comp
-L power:GNDREF #PWR043
-U 1 1 5D95D817
-P 1700 2950
-F 0 "#PWR043" H 1700 2700 50  0001 C CNN
-F 1 "GNDREF" H 1705 2777 50  0001 C CNN
-F 2 "" H 1700 2950 50  0001 C CNN
-F 3 "" H 1700 2950 50  0001 C CNN
-	1    1700 2950
-	1    0    0    -1
-$EndComp
 Text Label 1350 4050 0    50   ~ 0
 VCC1
@@
 VCC2
 Wire Wire Line
-	9350 3000 9350 3350
-Wire Wire Line
 	7550 3000 7550 3350
 Wire Wire Line
@@
 	6850 3750 6850 3900
 Connection ~ 5750 3900
-$Comp
-L power:GNDREF #PWR055
-U 1 1 5D8EF5E9
-P 8350 3950
-F 0 "#PWR055" H 8350 3700 50  0001 C CNN
-F 1 "GNDREF" H 8355 3777 50  0001 C CNN
-F 2 "" H 8350 3950 50  0001 C CNN
-F 3 "" H 8350 3950 50  0001 C CNN
-	1    8350 3950
-	1    0    0    -1
-$EndComp
 Wire Wire Line
 	6850 3900 7550 3900
@@
 	7550 3750 7550 3900
 Connection ~ 6850 3900
-Wire Wire Line
-	7550 3900 8350 3900
-Wire Wire Line
-	8350 3900 8350 3950
 Connection ~ 7550 3900
 Wire Wire Line
-	8350 3900 8750 3900
-Wire Wire Line
 	8750 3500 8750 3900
-Connection ~ 8350 3900
-Wire Wire Line
-	8750 3900 9350 3900
-Wire Wire Line
-	9350 3650 9350 3900
+Wire Wire Line
+	9600 3650 9600 3900
 Connection ~ 8750 3900
 Wire Wire Line
@@
 	1    0    0    -1
 $EndComp
+Wire Wire Line
+	4600 3000 5000 3000
+$Comp
+L power:PWR_FLAG #FLG0101
+U 1 1 5DBD1258
+P 5000 3000
+F 0 "#FLG0101" H 5000 3075 50  0001 C CNN
+F 1 "PWR_FLAG" H 5000 3173 50  0000 C CNN
+F 2 "" H 5000 3000 50  0001 C CNN
+F 3 "~" H 5000 3000 50  0001 C CNN
+	1    5000 3000
+	1    0    0    -1
+$EndComp
+Connection ~ 5000 3000
+Wire Wire Line
+	5000 3000 5250 3000
+$Comp
+L power:PWR_FLAG #FLG0102
+U 1 1 5DBD1EE4
+P 7200 3000
+F 0 "#FLG0102" H 7200 3075 50  0001 C CNN
+F 1 "PWR_FLAG" H 7200 3173 50  0000 C CNN
+F 2 "" H 7200 3000 50  0001 C CNN
+F 3 "~" H 7200 3000 50  0001 C CNN
+	1    7200 3000
+	1    0    0    -1
+$EndComp
+Connection ~ 7200 3000
+Wire Wire Line
+	7200 3000 7550 3000
+$Comp
+L power:PWR_FLAG #FLG0103
+U 1 1 5DBD2DF8
+P 9300 2950
+F 0 "#FLG0103" H 9300 3025 50  0001 C CNN
+F 1 "PWR_FLAG" H 9300 3123 50  0000 C CNN
+F 2 "" H 9300 2950 50  0001 C CNN
+F 3 "~" H 9300 2950 50  0001 C CNN
+	1    9300 2950
+	1    0    0    -1
+$EndComp
+Wire Wire Line
+	9600 2950 9600 3000
+Connection ~ 9600 3000
+Wire Wire Line
+	9600 3000 9600 3350
+Wire Wire Line
+	8750 3900 8950 3900
+Connection ~ 9300 3000
+Wire Wire Line
+	9300 3000 9250 3000
+Wire Wire Line
+	9300 3000 9600 3000
+Wire Wire Line
+	8550 3900 8550 3950
+Connection ~ 8550 3900
+Wire Wire Line
+	8550 3900 8750 3900
+$Comp
+L power:GND #PWR0103
+U 1 1 5DC523AE
+P 8950 3900
+F 0 "#PWR0103" H 8950 3650 50  0001 C CNN
+F 1 "GND" H 8955 3727 50  0000 C CNN
+F 2 "" H 8950 3900 50  0001 C CNN
+F 3 "" H 8950 3900 50  0001 C CNN
+	1    8950 3900
+	1    0    0    -1
+$EndComp
+$Comp
+L power:GND #PWR0104
+U 1 1 5DC52755
+P 1700 2950
+F 0 "#PWR0104" H 1700 2700 50  0001 C CNN
+F 1 "GND" H 1705 2777 50  0000 C CNN
+F 2 "" H 1700 2950 50  0001 C CNN
+F 3 "" H 1700 2950 50  0001 C CNN
+	1    1700 2950
+	1    0    0    -1
+$EndComp
+$Comp
+L power:GND #PWR0105
+U 1 1 5DC542C3
+P 1700 3900
+F 0 "#PWR0105" H 1700 3650 50  0001 C CNN
+F 1 "GND" H 1705 3727 50  0000 C CNN
+F 2 "" H 1700 3900 50  0001 C CNN
+F 3 "" H 1700 3900 50  0001 C CNN
+	1    1700 3900
+	1    0    0    -1
+$EndComp
+Wire Wire Line
+	1300 3850 1700 3850
+Wire Wire Line
+	1300 2900 1700 2900
+Connection ~ 8950 3900
+Wire Wire Line
+	8950 3900 9600 3900
+Wire Wire Line
+	7550 3900 8550 3900
+$Comp
+L power:PWR_FLAG #FLG?
+U 1 1 5DC68C13
+P 8550 3950
+F 0 "#FLG?" H 8550 4025 50  0001 C CNN
+F 1 "PWR_FLAG" H 8550 4123 50  0000 C CNN
+F 2 "" H 8550 3950 50  0001 C CNN
+F 3 "~" H 8550 3950 50  0001 C CNN
+	1    8550 3950
+	-1   0    0    1
+$EndComp
 $EndSCHEMATC

Commit message: Esquemático Finalizado. Asignaciones Realizadas. Comienzo de PCB.
Parts:
- C21, C22, C23: footprint (none) -> Capacitor_SMD:C_0805_2012Metric
- D1: footprint (none) -> LED_SMD:LED_0805_2012Metric
- D8: footprint (none) -> Diode_SMD:D_MiniMELF
- F1: footprint (none) -> Fuse:Fuse_0805_2012Metric
- J3, J4: footprint (none) -> Connector_PinSocket_1.27mm:PinSocket_1x04_P1.27mm_Vertical
- L1: footprint (none) -> Inductor_SMD:L_7.3x7.3_H4.5
- R9: footprint (none) -> Resistor_SMD:R_0805_2012Metric
Changed lines of the file:
@@
 F 0 "C21" H 5365 3496 50  0000 L CNN
 F 1 "22uF" H 5365 3405 50  0000 L CNN
-F 2 "" H 5288 3300 50  0001 C CNN
+F 2 "Capacitor_SMD:C_0805_2012Metric" H 5288 3300 50  0001 C CNN
 F 3 "~" H 5250 3450 50  0001 C CNN
 	1    5250 3450
@@
 F 0 "L1" V 7340 3350 50  0000 C CNN
 F 1 "330uH" V 7249 3350 50  0000 C CNN
-F 2 "" H 7150 3350 50  0001 C CNN
+F 2 "Inductor_SMD:L_7.3x7.3_H4.5" H 7150 3350 50  0001 C CNN
 F 3 "~" H 7150 3350 50  0001 C CNN
 	1    7150 3350
@@
 F 0 "D8" V 6804 3679 50  0000 L CNN
 F 1 "10MQ060N" V 6895 3679 50  0000 L CNN
-F 2 "" H 6850 3600 50  0001 C CNN
+F 2 "Diode_SMD:D_MiniMELF" H 6850 3600 50  0001 C CNN
 F 3 "~" H 6850 3600 50  0001 C CNN
 	1    6850 3600
@@
 F 0 "C22" H 7665 3646 50  0000 L CNN
 F 1 "220uF" H 7665 3555 50  0000 L CNN
-F 2 "" H 7588 3450 50  0001 C CNN
+F 2 "Capacitor_SMD:C_0805_2012Metric" H 7588 3450 50  0001 C CNN
 F 3 "~" H 7550 3600 50  0001 C CNN
 	1    7550 3600
@@
 F 0 "C23" H 9715 3546 50  0000 L CNN
 F 1 "10uF" H 9715 3455 50  0000 L CNN
-F 2 "" H 9638 3350 50  0001 C CNN
+F 2 "Capacitor_SMD:C_0805_2012Metric" H 9638 3350 50  0001 C CNN
 F 3 "~" H 9600 3500 50  0001 C CNN
 	1    9600 3500
@@
 F 0 "F1" V 3025 3250 50  0000 C CNN
 F 1 "Polyswitch" V 3116 3250 50  0000 C CNN
-F 2 "" H 3300 3050 50  0001 L CNN
+F 2 "Fuse:Fuse_0805_2012Metric" H 3300 3050 50  0001 L CNN
 F 3 "~" H 3250 3250 50  0001 C CNN
 	1    3250 3250
@@
 F 0 "D1" V 6689 4932 50  0000 R CNN
 F 1 "VCC_5V" V 6598 4932 50  0000 R CNN
-F 2 "" H 6650 5050 50  0001 C CNN
+F 2 "LED_SMD:LED_0805_2012Metric" H 6650 5050 50  0001 C CNN
 F 3 "~" H 6650 5050 50  0001 C CNN
 	1    6650 5050
@@
 F 0 "R9" H 6720 5446 50  0000 L CNN
 F 1 "470" H 6720 5355 50  0000 L CNN
-F 2 "" V 6580 5400 50  0001 C CNN
+F 2 "Resistor_SMD:R_0805_2012Metric" V 6580 5400 50  0001 C CNN
 F 3 "~" H 6650 5400 50  0001 C CNN
 	1    6650 5400
@@
 F 0 "J4" H 1208 4139 50  0000 C CNN
 F 1 "Conn_01x04_Male" H 1208 4140 50  0001 C CNN
-F 2 "" H 1100 3950 50  0001 C CNN
+F 2 "Connector_PinSocket_1.27mm:PinSocket_1x04_P1.27mm_Vertical" H 1100 3950 50  0001 C CNN
 F 3 "~" H 1100 3950 50  0001 C CNN
 	1    1100 3950
@@
 F 0 "J3" H 1208 3089 50  0000 C CNN
 F 1 "Conn_01x04_Male" H 1208 3090 50  0001 C CNN
-F 2 "" H 1100 2900 50  0001 C CNN
+F 2 "Connector_PinSocket_1.27mm:PinSocket_1x04_P1.27mm_Vertical" H 1100 2900 50  0001 C CNN
 F 3 "~" H 1100 2900 50  0001 C CNN
 	1    1100 2900
@@
 	7550 3900 8550 3900
 $Comp
-L power:PWR_FLAG #FLG?
+L power:PWR_FLAG #FLG0104
 U 1 1 5DC68C13
 P 8550 3950
-F 0 "#FLG?" H 8550 4025 50  0001 C CNN
+F 0 "#FLG0104" H 8550 4025 50  0001 C CNN
 F 1 "PWR_FLAG" H 8550 4123 50  0000 C CNN
 F 2 "" H 8550 3950 50  0001 C CNN

Commit message: Esquemático Finalizado. Asignaciones Realizadas. Componentes acomodados en PCB.
Parts:
- removed J3: Conn_01x04_Male, Connector_PinSocket_1.27mm:PinSocket_1x04_P1.27mm_Vertical, symbol Connector:Conn_01x04_Male
- renumbered C21 to C23, C22 to C24, C23 to C25, D2 to D5, D3 to D6, D1 to D7, J4 to J7, R9 to R8, U9 to U8, U10 to U9
Connections:
- net GNDREF is gone; now on net GND: R8.2
- net VCC1: now also J7.4 (Pin_4); no longer J7.3 (Pin_3)
- net VCC2: now also J7.3 (Pin_3); no longer J7.4 (Pin_4)
Changed lines of the file:
@@
 $EndDescr
 $Comp
-L Diode:BZT52Bxx D3
+L Diode:BZT52Bxx D6
 U 1 1 5D8AAC6F
 P 4600 3450
-F 0 "D3" V 4700 3500 50  0000 L CNN
+F 0 "D6" V 4700 3500 50  0000 L CNN
 F 1 "BZT52BC30-7" V 4800 3450 50  0000 L CNN
 F 2 "Diode_SMD:D_SOD-123" H 4600 3275 50  0001 C CNN
@@
 $EndComp
 $Comp
-L Device:C C21
+L Device:C C23
 U 1 1 5D8AC03F
 P 5250 3450
-F 0 "C21" H 5365 3496 50  0000 L CNN
+F 0 "C23" H 5365 3496 50  0000 L CNN
 F 1 "22uF" H 5365 3405 50  0000 L CNN
 F 2 "Capacitor_SMD:C_0805_2012Metric" H 5288 3300 50  0001 C CNN
@@
 $EndComp
 $Comp
-L Regulator_Switching:LM2574M-5 U9
+L Regulator_Switching:LM2574M-5 U8
 U 1 1 5D8ACF78
 P 6250 3100
-F 0 "U9" H 6250 3467 50  0000 C CNN
+F 0 "U8" H 6250 3467 50  0000 C CNN
 F 1 "LM2574M-5" H 6250 3376 50  0000 C CNN
 F 2 "Package_SO:SOIC-14W_7.5x9mm_P1.27mm" H 5850 3450 50  0001 L CIN
@@
 $EndComp
 $Comp
-L power:VCC #PWR049
+L power:VCC #PWR043
 U 1 1 5D8AF9E9
 P 4600 3000
-F 0 "#PWR049" H 4600 2850 50  0001 C CNN
+F 0 "#PWR043" H 4600 2850 50  0001 C CNN
 F 1 "VCC" H 4617 3173 50  0000 C CNN
 F 2 "" H 4600 3000 50  0001 C CNN
@@
 $EndComp
 $Comp
-L Device:C C22
+L Device:C C24
 U 1 1 5D8B1698
 P 7550 3600
-F 0 "C22" H 7665 3646 50  0000 L CNN
+F 0 "C24" H 7665 3646 50  0000 L CNN
 F 1 "220uF" H 7665 3555 50  0000 L CNN
 F 2 "Capacitor_SMD:C_0805_2012Metric" H 7588 3450 50  0001 C CNN
@@
 $EndComp
 $Comp
-L REG1117:REG1117 U10
+L REG1117:REG1117 U?
 U 1 1 5D8B1D75
 P 8750 3000
-AR Path="/5D8B1D75" Ref="U10"  Part="1"
-AR Path="/5D9FFB34/5D8B1D75" Ref="U10"  Part="1"
-F 0 "U10" H 8750 3370 50  0000 C CNN
+AR Path="/5D8B1D75" Ref="U?"  Part="1"
+AR Path="/5D9FFB34/5D8B1D75" Ref="U9"  Part="1"
+F 0 "U9" H 8750 3370 50  0000 C CNN
 F 1 "REG1117" H 8750 3279 50  0000 C CNN
 F 2 "REG1117:DD-3" H 8750 3000 50  0001 C CNN
@@
 $EndComp
 $Comp
-L Device:C C23
+L Device:C C25
 U 1 1 5D8B2AEE
 P 9600 3500
-F 0 "C23" H 9715 3546 50  0000 L CNN
+F 0 "C25" H 9715 3546 50  0000 L CNN
 F 1 "10uF" H 9715 3455 50  0000 L CNN
 F 2 "Capacitor_SMD:C_0805_2012Metric" H 9638 3350 50  0001 C CNN
@@
 $EndComp
 $Comp
-L Diode_Bridge:MB2S D2
+L Diode_Bridge:MB2S D5
 U 1 1 5D8AA31B
 P 4050 3550
-F 0 "D2" H 3900 3700 50  0000 R CNN
+F 0 "D5" H 3900 3700 50  0000 R CNN
 F 1 "MB2S" H 3950 3800 50  0000 R CNN
 F 2 "Package_TO_SOT_SMD:TO-269AA" H 4200 3675 50  0001 L CNN
@@
 Connection ~ 7550 3000
 $Comp
-L power:+3.3V #PWR058
+L power:+3.3V #PWR048
 U 1 1 5D8D85F9
 P 9600 2950
-F 0 "#PWR058" H 9600 2800 50  0001 C CNN
+F 0 "#PWR048" H 9600 2800 50  0001 C CNN
 F 1 "+3.3V" H 9615 3123 50  0000 C CNN
 F 2 "" H 9600 2950 50  0001 C CNN
@@
 	9300 3000 9300 2950
 $Comp
-L power:+5V #PWR054
+L power:+5V #PWR046
 U 1 1 5D8D958A
 P 7550 2950
-F 0 "#PWR054" H 7550 2800 50  0001 C CNN
+F 0 "#PWR046" H 7550 2800 50  0001 C CNN
 F 1 "+5V" H 7565 3123 50  0000 C CNN
 F 2 "" H 7550 2950 50  0001 C CNN
@@
 $EndComp
 $Comp
-L power:GNDREF #PWR046
-U 1 1 5D8EE8DF
-P 6650 5600
-F 0 "#PWR046" H 6650 5350 50  0001 C CNN
-F 1 "GNDREF" H 6655 5427 50  0001 C CNN
-F 2 "" H 6650 5600 50  0001 C CNN
-F 3 "" H 6650 5600 50  0001 C CNN
-	1    6650 5600
-	1    0    0    -1
-$EndComp
-$Comp
-L Device:LED_ALT D1
+L Device:LED_ALT D7
 U 1 1 5D8FBCC8
 P 6650 5050
-F 0 "D1" V 6689 4932 50  0000 R CNN
+F 0 "D7" V 6689 4932 50  0000 R CNN
 F 1 "VCC_5V" V 6598 4932 50  0000 R CNN
 F 2 "LED_SMD:LED_0805_2012Metric" H 6650 5050 50  0001 C CNN
@@
 $EndComp
 $Comp
-L Device:R R9
+L Device:R R8
 U 1 1 5D8FD671
 P 6650 5400
-F 0 "R9" H 6720 5446 50  0000 L CNN
+F 0 "R8" H 6720 5446 50  0000 L CNN
 F 1 "470" H 6720 5355 50  0000 L CNN
 F 2 "Resistor_SMD:R_0805_2012Metric" V 6580 5400 50  0001 C CNN
@@
 Connection ~ 1300 3850
 $Comp
-L Connector:Conn_01x04_Male J4
+L Connector:Conn_01x04_Male J7
 U 1 1 5D93EED0
 P 1100 3950
-F 0 "J4" H 1208 4139 50  0000 C CNN
+F 0 "J7" H 1208 4139 50  0000 C CNN
 F 1 "Conn_01x04_Male" H 1208 4140 50  0001 C CNN
 F 2 "Connector_PinSocket_1.27mm:PinSocket_1x04_P1.27mm_Vertical" H 1100 3950 50  0001 C CNN
@@
 	1    0    0    -1
 $EndComp
-$Comp
-L Connector:Conn_01x04_Male J3
-U 1 1 5D93E22F
-P 1100 2900
-F 0 "J3" H 1208 3089 50  0000 C CNN
-F 1 "Conn_01x04_Male" H 1208 3090 50  0001 C CNN
-F 2 "Connector_PinSocket_1.27mm:PinSocket_1x04_P1.27mm_Vertical" H 1100 2900 50  0001 C CNN
-F 3 "~" H 1100 2900 50  0001 C CNN
-	1    1100 2900
-	1    0    0    -1
-$EndComp
-Connection ~ 1300 3000
-Wire Wire Line
-	1300 3000 1300 3100
-Wire Wire Line
-	1300 2900 1300 3000
-Wire Wire Line
-	1300 2800 1300 2900
-Connection ~ 1300 2900
-Wire Wire Line
-	1700 2900 1700 2950
+Text Label 1350 4150 0    50   ~ 0
+VCC1
 Text Label 1350 4050 0    50   ~ 0
-VCC1
-Text Label 1350 4150 0    50   ~ 0
 VCC2
 Text Label 3000 3250 2    50   ~ 0
@@
 	7550 3750 7550 3900
 Connection ~ 6850 3900
-Connection ~ 7550 3900
 Wire Wire Line
 	8750 3500 8750 3900
@@
 	6650 4750 6650 4900
 $Comp
-L power:+5V #PWR0101
+L power:+5V #PWR044
 U 1 1 5DBD8410
 P 6650 4750
-F 0 "#PWR0101" H 6650 4600 50  0001 C CNN
+F 0 "#PWR044" H 6650 4600 50  0001 C CNN
 F 1 "+5V" H 6665 4923 50  0000 C CNN
 F 2 "" H 6650 4750 50  0001 C CNN
@@
 	4600 3000 5000 3000
 $Comp
-L power:PWR_FLAG #FLG0101
+L power:PWR_FLAG #FLG01
 U 1 1 5DBD1258
 P 5000 3000
-F 0 "#FLG0101" H 5000 3075 50  0001 C CNN
+F 0 "#FLG01" H 5000 3075 50  0001 C CNN
 F 1 "PWR_FLAG" H 5000 3173 50  0000 C CNN
 F 2 "" H 5000 3000 50  0001 C CNN
@@
 	5000 3000 5250 3000
 $Comp
-L power:PWR_FLAG #FLG0102
+L power:PWR_FLAG #FLG02
 U 1 1 5DBD1EE4
 P 7200 3000
-F 0 "#FLG0102" H 7200 3075 50  0001 C CNN
+F 0 "#FLG02" H 7200 3075 50  0001 C CNN
 F 1 "PWR_FLAG" H 7200 3173 50  0000 C CNN
 F 2 "" H 7200 3000 50  0001 C CNN
@@
 	7200 3000 7550 3000
 $Comp
-L power:PWR_FLAG #FLG0103
+L power:PWR_FLAG #FLG03
 U 1 1 5DBD2DF8
 P 9300 2950
-F 0 "#FLG0103" H 9300 3025 50  0001 C CNN
+F 0 "#FLG03" H 9300 3025 50  0001 C CNN
 F 1 "PWR_FLAG" H 9300 3123 50  0000 C CNN
 F 2 "" H 9300 2950 50  0001 C CNN
@@
 Wire Wire Line
 	9300 3000 9600 3000
-Wire Wire Line
-	8550 3900 8550 3950
-Connection ~ 8550 3900
-Wire Wire Line
-	8550 3900 8750 3900
-$Comp
-L power:GND #PWR0103
+$Comp
+L power:GND #PWR047
 U 1 1 5DC523AE
 P 8950 3900
-F 0 "#PWR0103" H 8950 3650 50  0001 C CNN
+F 0 "#PWR047" H 8950 3650 50  0001 C CNN
 F 1 "GND" H 8955 3727 50  0000 C CNN
 F 2 "" H 8950 3900 50  0001 C CNN
@@
 $EndComp
 $Comp
-L power:GND #PWR0104
-U 1 1 5DC52755
-P 1700 2950
-F 0 "#PWR0104" H 1700 2700 50  0001 C CNN
-F 1 "GND" H 1705 2777 50  0000 C CNN
-F 2 "" H 1700 2950 50  0001 C CNN
-F 3 "" H 1700 2950 50  0001 C CNN
-	1    1700 2950
-	1    0    0    -1
-$EndComp
-$Comp
-L power:GND #PWR0105
+L power:GND #PWR042
 U 1 1 5DC542C3
 P 1700 3900
-F 0 "#PWR0105" H 1700 3650 50  0001 C CNN
+F 0 "#PWR042" H 1700 3650 50  0001 C CNN
 F 1 "GND" H 1705 3727 50  0000 C CNN
 F 2 "" H 1700 3900 50  0001 C CNN
@@
 Wire Wire Line
 	1300 3850 1700 3850
-Wire Wire Line
-	1300 2900 1700 2900
 Connection ~ 8950 3900
 Wire Wire Line
 	8950 3900 9600 3900
-Wire Wire Line
-	7550 3900 8550 3900
-$Comp
-L power:PWR_FLAG #FLG0104
-U 1 1 5DC68C13
-P 8550 3950
-F 0 "#FLG0104" H 8550 4025 50  0001 C CNN
-F 1 "PWR_FLAG" H 8550 4123 50  0000 C CNN
-F 2 "" H 8550 3950 50  0001 C CNN
-F 3 "~" H 8550 3950 50  0001 C CNN
-	1    8550 3950
+$Comp
+L power:GND #PWR045
+U 1 1 5DC8CD17
+P 6650 5600
+F 0 "#PWR045" H 6650 5350 50  0001 C CNN
+F 1 "GND" H 6655 5427 50  0000 C CNN
+F 2 "" H 6650 5600 50  0001 C CNN
+F 3 "" H 6650 5600 50  0001 C CNN
+	1    6650 5600
+	1    0    0    -1
+$EndComp
+Wire Wire Line
+	7550 3900 8350 3900
+Connection ~ 7550 3900
+$Comp
+L power:PWR_FLAG #FLG0101
+U 1 1 5DCD1DAC
+P 8350 3900
+F 0 "#FLG0101" H 8350 3975 50  0001 C CNN
+F 1 "PWR_FLAG" H 8350 4073 50  0000 C CNN
+F 2 "" H 8350 3900 50  0001 C CNN
+F 3 "~" H 8350 3900 50  0001 C CNN
+	1    8350 3900
 	-1   0    0    1
 $EndComp
+Connection ~ 8350 3900
+Wire Wire Line
+	8350 3900 8750 3900
 $EndSCHEMATC
