File: Bridge_Ethernet/Micro.sch (KiCad schematic (older format))
At the start: 11 parts, among them J7 Conn_2Rows-13Pins, U13 MSP430F5438A

Commit message: Esquemático Finalizado, sin warnings. Haciendo asignaciones de footprints
Changed lines of the file:
@@
 L power:GND #PWR070
 U 1 1 5D9672BE
-P 1500 4150
-F 0 "#PWR070" H 1500 3900 50  0001 C CNN
-F 1 "GND" H 1505 3977 50  0000 C CNN
-F 2 "" H 1500 4150 50  0001 C CNN
-F 3 "" H 1500 4150 50  0001 C CNN
-	1    1500 4150
+P 1500 4000
+F 0 "#PWR070" H 1500 3750 50  0001 C CNN
+F 1 "GND" H 1505 3827 50  0000 C CNN
+F 2 "" H 1500 4000 50  0001 C CNN
+F 3 "" H 1500 4000 50  0001 C CNN
+	1    1500 4000
 	1    0    0    -1
 $EndComp
@@
 Wire Wire Line
 	1500 3600 1500 4000
-Connection ~ 1500 4000
-Wire Wire Line
-	1500 4000 1500 4150
 Wire Wire Line
 	1800 4000 1500 4000
@@
 L power:GND #PWR077
 U 1 1 5D97C24F
-P 5300 3850
-F 0 "#PWR077" H 5300 3600 50  0001 C CNN
-F 1 "GND" H 5305 3677 50  0000 C CNN
-F 2 "" H 5300 3850 50  0001 C CNN
-F 3 "" H 5300 3850 50  0001 C CNN
-	1    5300 3850
-	-1   0    0    -1
-$EndComp
-Wire Wire Line
-	5300 3850 5300 3800
+P 4950 3800
+F 0 "#PWR077" H 4950 3550 50  0001 C CNN
+F 1 "GND" H 4955 3627 50  0000 C CNN
+F 2 "" H 4950 3800 50  0001 C CNN
+F 3 "" H 4950 3800 50  0001 C CNN
+	1    4950 3800
+	-1   0    0    -1
+$EndComp
 Wire Wire Line
 	4650 3400 4950 3400
@@
 Wire Wire Line
 	4950 3800 5300 3800
-Connection ~ 5300 3800
 $Comp
 L Device:C C36
@@
 L power:GND #PWR082
 U 1 1 5DA67B8D
-P 7550 2950
-F 0 "#PWR082" H 7550 2700 50  0001 C CNN
-F 1 "GND" H 7555 2777 50  0000 C CNN
-F 2 "" H 7550 2950 50  0001 C CNN
-F 3 "" H 7550 2950 50  0001 C CNN
-	1    7550 2950
-	-1   0    0    -1
-$EndComp
-Wire Wire Line
-	7200 2850 7550 2850
-Wire Wire Line
-	7550 2850 7550 2950
+P 7400 2850
+F 0 "#PWR082" H 7400 2600 50  0001 C CNN
+F 1 "GND" H 7405 2677 50  0000 C CNN
+F 2 "" H 7400 2850 50  0001 C CNN
+F 3 "" H 7400 2850 50  0001 C CNN
+	1    7400 2850
+	-1   0    0    -1
+$EndComp
+Wire Wire Line
+	7200 2850 7400 2850
 $Comp
 L Device:R R12
@@
 NoConn ~ 6700 2650
 NoConn ~ 6700 2850
+Connection ~ 4950 3800
+Connection ~ 1500 4000
 $EndSCHEMATC

Commit message: Esquemático Finalizado. Asignaciones Realizadas. Comienzo de PCB.
Parts:
- C30, C31, C32, C33, C34, C35, C36, C37: footprint (none) -> Capacitor_SMD:C_0805_2012Metric
- J7: footprint (none) -> Connector_PinHeader_1.27mm:PinHeader_2x07_P1.27mm_Vertical
- R12: footprint (none) -> Resistor_SMD:R_0805_2012Metric
- U13: footprint PZ100 -> MSP430F5438A:PZ100
Changed lines of the file:
@@
 F 0 "U13" H 3475 7665 50  0000 C CNN
 F 1 "MSP430F5438A" H 7950 5700 50  0001 L BNN
-F 2 "PZ100" H 6900 5650 50  0001 L BNN
+F 2 "MSP430F5438A:PZ100" H 6900 5650 50  0001 L BNN
 F 3 "Texas Instruments" H 7950 5800 50  0001 L BNN
 F 4 "16-bit ultra-low-power microcontroller, 256kb flash, 16kb ram, 12 bit adc, 4 uscis, 32-bit hw multi" H 7300 5550 50  0001 L BNN "Field4"
@@
 F 0 "C33" V 2000 3550 50  0000 C CNN
 F 1 "0.1uF" V 2100 3550 50  0000 C CNN
-F 2 "" H 2088 3250 50  0001 C CNN
+F 2 "Capacitor_SMD:C_0805_2012Metric" H 2088 3250 50  0001 C CNN
 F 3 "~" H 2050 3400 50  0001 C CNN
 	1    2050 3400
@@
 F 0 "C30" H 1400 3050 50  0000 C CNN
 F 1 "0.1uF" H 1650 3050 50  0000 C CNN
-F 2 "" H 1538 3000 50  0001 C CNN
+F 2 "Capacitor_SMD:C_0805_2012Metric" H 1538 3000 50  0001 C CNN
 F 3 "~" H 1500 3150 50  0001 C CNN
 	1    1500 3150
@@
 F 0 "C32" H 1700 3950 50  0000 C CNN
 F 1 "0.1uF" H 1700 3750 50  0000 C CNN
-F 2 "" H 1838 3700 50  0001 C CNN
+F 2 "Capacitor_SMD:C_0805_2012Metric" H 1838 3700 50  0001 C CNN
 F 3 "~" H 1800 3850 50  0001 C CNN
 	1    1800 3850
@@
 F 0 "C31" H 1750 6150 50  0000 C CNN
 F 1 "0.1uF" H 1800 5950 50  0000 C CNN
-F 2 "" H 1688 5900 50  0001 C CNN
+F 2 "Capacitor_SMD:C_0805_2012Metric" H 1688 5900 50  0001 C CNN
 F 3 "~" H 1650 6050 50  0001 C CNN
 	1    1650 6050
@@
 F 0 "C35" H 5200 3750 50  0000 C CNN
 F 1 "0.1uF" H 5150 3550 50  0000 C CNN
-F 2 "" H 5338 3500 50  0001 C CNN
+F 2 "Capacitor_SMD:C_0805_2012Metric" H 5338 3500 50  0001 C CNN
 F 3 "~" H 5300 3650 50  0001 C CNN
 	1    5300 3650
@@
 F 0 "C36" H 5200 6050 50  0000 C CNN
 F 1 "0.1uF" H 5150 5850 50  0000 C CNN
-F 2 "" H 5338 5800 50  0001 C CNN
+F 2 "Capacitor_SMD:C_0805_2012Metric" H 5338 5800 50  0001 C CNN
 F 3 "~" H 5300 5950 50  0001 C CNN
 	1    5300 5950
@@
 F 0 "C34" H 4750 6250 50  0000 C CNN
 F 1 "470nF" H 4700 6050 50  0000 C CNN
-F 2 "" H 4888 6000 50  0001 C CNN
+F 2 "Capacitor_SMD:C_0805_2012Metric" H 4888 6000 50  0001 C CNN
 F 3 "~" H 4850 6150 50  0001 C CNN
 	1    4850 6150
@@
 F 0 "J7" H 6950 3267 50  0000 C CNN
 F 1 "Conn_2Rows-13Pins" H 6950 3176 50  0000 C CNN
-F 2 "" H 6900 2750 50  0001 C CNN
+F 2 "Connector_PinHeader_1.27mm:PinHeader_2x07_P1.27mm_Vertical" H 6900 2750 50  0001 C CNN
 F 3 "~" H 6900 2750 50  0001 C CNN
 	1    6900 2750
@@
 F 0 "R12" H 7270 3796 50  0000 L CNN
 F 1 "47K" H 7270 3705 50  0000 L CNN
-F 2 "" V 7130 3750 50  0001 C CNN
+F 2 "Resistor_SMD:R_0805_2012Metric" V 7130 3750 50  0001 C CNN
 F 3 "~" H 7200 3750 50  0001 C CNN
 	1    7200 3750
@@
 F 0 "C37" H 7100 4250 50  0000 C CNN
 F 1 "0.1uF" H 7050 4050 50  0000 C CNN
-F 2 "" H 7238 4000 50  0001 C CNN
+F 2 "Capacitor_SMD:C_0805_2012Metric" H 7238 4000 50  0001 C CNN
 F 3 "~" H 7200 4150 50  0001 C CNN
 	1    7200 4150

Commit message: Esquemático Finalizado. Asignaciones Realizadas. Componentes acomodados en PCB.
Parts:
- renumbered C30 to C15, C31 to C16, C32 to C17, C33 to C18, C34 to C19, C35 to C20, C36 to C21, C37 to C22, J7 to J5, R12 to R7, U13 to U7
Changed lines of the file:
@@
 $EndDescr
 $Comp
-L MSP430F5438A:MSP430F5438A U13
+L MSP430F5438A:MSP430F5438A U?
 U 1 1 5D952D6C
 P 3500 4700
-AR Path="/5D952D6C" Ref="U13"  Part="1"
-AR Path="/5DA0E37F/5D952D6C" Ref="U13"  Part="1"
-F 0 "U13" H 3475 7665 50  0000 C CNN
+AR Path="/5D952D6C" Ref="U?"  Part="1"
+AR Path="/5DA0E37F/5D952D6C" Ref="U7"  Part="1"
+F 0 "U7" H 3475 7665 50  0000 C CNN
 F 1 "MSP430F5438A" H 7950 5700 50  0001 L BNN
 F 2 "MSP430F5438A:PZ100" H 6900 5650 50  0001 L BNN
@@
 NoConn ~ 4650 3200
 $Comp
-L Device:C C33
+L Device:C C18
 U 1 1 5D95FA2D
 P 2050 3400
-F 0 "C33" V 2000 3550 50  0000 C CNN
+F 0 "C18" V 2000 3550 50  0000 C CNN
 F 1 "0.1uF" V 2100 3550 50  0000 C CNN
 F 2 "Capacitor_SMD:C_0805_2012Metric" H 2088 3250 50  0001 C CNN
@@
 	2200 3200 2300 3200
 $Comp
-L Device:C C30
+L Device:C C15
 U 1 1 5D965F8F
 P 1500 3150
-F 0 "C30" H 1400 3050 50  0000 C CNN
+F 0 "C15" H 1400 3050 50  0000 C CNN
 F 1 "0.1uF" H 1650 3050 50  0000 C CNN
 F 2 "Capacitor_SMD:C_0805_2012Metric" H 1538 3000 50  0001 C CNN
@@
 $EndComp
 $Comp
-L power:GND #PWR070
+L power:GND #PWR030
 U 1 1 5D9672BE
 P 1500 4000
-F 0 "#PWR070" H 1500 3750 50  0001 C CNN
+F 0 "#PWR030" H 1500 3750 50  0001 C CNN
 F 1 "GND" H 1505 3827 50  0000 C CNN
 F 2 "" H 1500 4000 50  0001 C CNN
@@
 $EndComp
 $Comp
-L power:+3V3 #PWR069
+L power:+3V3 #PWR029
 U 1 1 5D967AF1
 P 1500 2950
-F 0 "#PWR069" H 1500 2800 50  0001 C CNN
+F 0 "#PWR029" H 1500 2800 50  0001 C CNN
 F 1 "+3V3" H 1515 3123 50  0000 C CNN
 F 2 "" H 1500 2950 50  0001 C CNN
@@
 Connection ~ 1500 3600
 $Comp
-L Device:C C32
+L Device:C C17
 U 1 1 5D96B207
 P 1800 3850
-F 0 "C32" H 1700 3950 50  0000 C CNN
+F 0 "C17" H 1700 3950 50  0000 C CNN
 F 1 "0.1uF" H 1700 3750 50  0000 C CNN
 F 2 "Capacitor_SMD:C_0805_2012Metric" H 1838 3700 50  0001 C CNN
@@
 	1800 3000 2200 3000
 $Comp
-L Device:C C31
+L Device:C C16
 U 1 1 5D975AF3
 P 1650 6050
-F 0 "C31" H 1750 6150 50  0000 C CNN
+F 0 "C16" H 1750 6150 50  0000 C CNN
 F 1 "0.1uF" H 1800 5950 50  0000 C CNN
 F 2 "Capacitor_SMD:C_0805_2012Metric" H 1688 5900 50  0001 C CNN
@@
 $EndComp
 $Comp
-L power:+3V3 #PWR073
+L power:+3V3 #PWR031
 U 1 1 5D975AF9
 P 1650 5850
-F 0 "#PWR073" H 1650 5700 50  0001 C CNN
+F 0 "#PWR031" H 1650 5700 50  0001 C CNN
 F 1 "+3V3" H 1665 6023 50  0000 C CNN
 F 2 "" H 1650 5850 50  0001 C CNN
@@
 	1650 5900 2300 5900
 $Comp
-L power:GND #PWR074
+L power:GND #PWR032
 U 1 1 5D976D7D
 P 1650 6250
-F 0 "#PWR074" H 1650 6000 50  0001 C CNN
+F 0 "#PWR032" H 1650 6000 50  0001 C CNN
 F 1 "GND" H 1655 6077 50  0000 C CNN
 F 2 "" H 1650 6250 50  0001 C CNN
@@
 $EndComp
 $Comp
-L Device:C C35
+L Device:C C20
 U 1 1 5D97C240
 P 5300 3650
-F 0 "C35" H 5200 3750 50  0000 C CNN
+F 0 "C20" H 5200 3750 50  0000 C CNN
 F 1 "0.1uF" H 5150 3550 50  0000 C CNN
 F 2 "Capacitor_SMD:C_0805_2012Metric" H 5338 3500 50  0001 C CNN
@@
 $EndComp
 $Comp
-L power:+3V3 #PWR076
+L power:+3V3 #PWR035
 U 1 1 5D97C246
 P 5300 3450
-F 0 "#PWR076" H 5300 3300 50  0001 C CNN
+F 0 "#PWR035" H 5300 3300 50  0001 C CNN
 F 1 "+3V3" H 5315 3623 50  0000 C CNN
 F 2 "" H 5300 3450 50  0001 C CNN
@@
 	5300 3500 4650 3500
 $Comp
-L power:GND #PWR077
+L power:GND #PWR034
 U 1 1 5D97C24F
 P 4950 3800
-F 0 "#PWR077" H 4950 3550 50  0001 C CNN
+F 0 "#PWR034" H 4950 3550 50  0001 C CNN
 F 1 "GND" H 4955 3627 50  0000 C CNN
 F 2 "" H 4950 3800 50  0001 C CNN
@@
 	4950 3800 5300 3800
 $Comp
-L Device:C C36
+L Device:C C21
 U 1 1 5D988D2A
 P 5300 5950
-F 0 "C36" H 5200 6050 50  0000 C CNN
+F 0 "C21" H 5200 6050 50  0000 C CNN
 F 1 "0.1uF" H 5150 5850 50  0000 C CNN
 F 2 "Capacitor_SMD:C_0805_2012Metric" H 5338 5800 50  0001 C CNN
@@
 $EndComp
 $Comp
-L power:+3V3 #PWR078
+L power:+3V3 #PWR036
 U 1 1 5D988D30
 P 5300 5750
-F 0 "#PWR078" H 5300 5600 50  0001 C CNN
+F 0 "#PWR036" H 5300 5600 50  0001 C CNN
 F 1 "+3V3" H 5315 5923 50  0000 C CNN
 F 2 "" H 5300 5750 50  0001 C CNN
@@
 	5300 5800 4650 5800
 $Comp
-L power:GND #PWR079
+L power:GND #PWR037
 U 1 1 5D988D39
 P 5300 6150
-F 0 "#PWR079" H 5300 5900 50  0001 C CNN
+F 0 "#PWR037" H 5300 5900 50  0001 C CNN
 F 1 "GND" H 5305 5977 50  0000 C CNN
 F 2 "" H 5300 6150 50  0001 C CNN
@@
 Connection ~ 5300 6100
 $Comp
-L Device:C C34
+L Device:C C19
 U 1 1 5D98B221
 P 4850 6150
-F 0 "C34" H 4750 6250 50  0000 C CNN
+F 0 "C19" H 4750 6250 50  0000 C CNN
 F 1 "470nF" H 4700 6050 50  0000 C CNN
 F 2 "Capacitor_SMD:C_0805_2012Metric" H 4888 6000 50  0001 C CNN
@@
 $EndComp
 $Comp
-L power:GND #PWR075
+L power:GND #PWR033
 U 1 1 5D98B230
 P 4850 6350
-F 0 "#PWR075" H 4850 6100 50  0001 C CNN
+F 0 "#PWR033" H 4850 6100 50  0001 C CNN
 F 1 "GND" H 4855 6177 50  0000 C CNN
 F 2 "" H 4850 6350 50  0001 C CNN
@@
 	4650 4200 4750 4200
 $Comp
-L Connector_Generic:Conn_2Rows-13Pins J7
+L Connector_Generic:Conn_2Rows-13Pins J5
 U 1 1 5DA22BBC
 P 6900 2750
-F 0 "J7" H 6950 3267 50  0000 C CNN
+F 0 "J5" H 6950 3267 50  0000 C CNN
 F 1 "Conn_2Rows-13Pins" H 6950 3176 50  0000 C CNN
 F 2 "Connector_PinHeader_1.27mm:PinHeader_2x07_P1.27mm_Vertical" H 6900 2750 50  0001 C CNN
@@
 	6650 3050 6700 3050
 $Comp
-L power:GND #PWR082
+L power:GND #PWR040
 U 1 1 5DA67B8D
 P 7400 2850
-F 0 "#PWR082" H 7400 2600 50  0001 C CNN
+F 0 "#PWR040" H 7400 2600 50  0001 C CNN
 F 1 "GND" H 7405 2677 50  0000 C CNN
 F 2 "" H 7400 2850 50  0001 C CNN
@@
 	7200 2850 7400 2850
 $Comp
-L Device:R R12
+L Device:R R7
 U 1 1 5DA69499
 P 7200 3750
-F 0 "R12" H 7270 3796 50  0000 L CNN
+F 0 "R7" H 7270 3796 50  0000 L CNN
 F 1 "47K" H 7270 3705 50  0000 L CNN
 F 2 "Resistor_SMD:R_0805_2012Metric" V 7130 3750 50  0001 C CNN
@@
 	7200 2950 7200 3400
 $Comp
-L power:+3V3 #PWR080
+L power:+3V3 #PWR038
 U 1 1 5DA6BEAE
 P 6900 3850
-F 0 "#PWR080" H 6900 3700 50  0001 C CNN
+F 0 "#PWR038" H 6900 3700 50  0001 C CNN
 F 1 "+3V3" H 6915 4023 50  0000 C CNN
 F 2 "" H 6900 3850 50  0001 C CNN
@@
 	6900 3900 7200 3900
 $Comp
-L Device:C C37
+L Device:C C22
 U 1 1 5DA6D954
 P 7200 4150
-F 0 "C37" H 7100 4250 50  0000 C CNN
+F 0 "C22" H 7100 4250 50  0000 C CNN
 F 1 "0.1uF" H 7050 4050 50  0000 C CNN
 F 2 "Capacitor_SMD:C_0805_2012Metric" H 7238 4000 50  0001 C CNN
@@
 Connection ~ 7200 3900
 $Comp
-L power:GND #PWR081
+L power:GND #PWR039
 U 1 1 5DA6F24D
 P 7200 4400
-F 0 "#PWR081" H 7200 4150 50  0001 C CNN
+F 0 "#PWR039" H 7200 4150 50  0001 C CNN
 F 1 "GND" H 7205 4227 50  0000 C CNN
 F 2 "" H 7200 4400 50  0001 C CNN
