File: Bridge_Ethernet/Bridge_Ethernet.sch (KiCad schematic (older format))
At the start: 2 parts, among them J5 Conn_01x04_Female, J6 Conn_01x04_Female

Commit message: Esquemático Finalizado. Asignaciones Realizadas. Comienzo de PCB.
Parts:
- J5, J6: footprint (none) -> Connector_PinSocket_1.27mm:PinSocket_1x04_P1.27mm_Vertical
Changed lines of the file:
@@
 F 0 "J5" H 778 3230 50  0000 L CNN
 F 1 "Conn_01x04_Female" H 778 3185 50  0001 L CNN
-F 2 "" H 750 3300 50  0001 C CNN
+F 2 "Connector_PinSocket_1.27mm:PinSocket_1x04_P1.27mm_Vertical" H 750 3300 50  0001 C CNN
 F 3 "~" H 750 3300 50  0001 C CNN
 	1    750  3300
@@
 F 0 "J6" H 828 4280 50  0000 L CNN
 F 1 "Conn_01x04_Female" H 828 4235 50  0001 L CNN
-F 2 "" H 800 4350 50  0001 C CNN
+F 2 "Connector_PinSocket_1.27mm:PinSocket_1x04_P1.27mm_Vertical" H 800 4350 50  0001 C CNN
 F 3 "~" H 800 4350 50  0001 C CNN
 	1    800  4350

Commit message: Esquemático Finalizado. Asignaciones Realizadas. Componentes acomodados en PCB.
Parts:
- renumbered J5 to J1, J6 to J2
Changed lines of the file:
@@
 P 750 3300
 AR Path="/5D9FFB34/5DBF2B33" Ref="J?"  Part="1"
-AR Path="/5DBF2B33" Ref="J5"  Part="1"
-F 0 "J5" H 778 3230 50  0000 L CNN
+AR Path="/5DBF2B33" Ref="J1"  Part="1"
+F 0 "J1" H 778 3230 50  0000 L CNN
 F 1 "Conn_01x04_Female" H 778 3185 50  0001 L CNN
 F 2 "Connector_PinSocket_1.27mm:PinSocket_1x04_P1.27mm_Vertical" H 750 3300 50  0001 C CNN
@@
 P 800 4350
 AR Path="/5D9FFB34/5DBF2B39" Ref="J?"  Part="1"
-AR Path="/5DBF2B39" Ref="J6"  Part="1"
-F 0 "J6" H 828 4280 50  0000 L CNN
+AR Path="/5DBF2B39" Ref="J2"  Part="1"
+F 0 "J2" H 828 4280 50  0000 L CNN
 F 1 "Conn_01x04_Female" H 828 4235 50  0001 L CNN
 F 2 "Connector_PinSocket_1.27mm:PinSocket_1x04_P1.27mm_Vertical" H 800 4350 50  0001 C CNN

Commit message: v2.0. Faltan algunos componentes 3D. Correciones relizadas.
Parts:
- added H1, H2, H3, H4: MountingHole, MountingHole:MountingHole_2.5mm_Pad, symbol Mechanical:MountingHole
Changed lines of the file:
@@
 Rev "Bridge Ethernet"
 Comp "Leandro Torrent"
-Comment1 ""
+Comment1 "Revisores: Martín Ribelotta, Miguel del Valle Camino"
 Comment2 ""
 Comment3 ""
@@
 Text Label 8700 5250 2    50   ~ 0
 RX_232_3
+$Comp
+L Mechanical:MountingHole H1
+U 1 1 5DD37999
+P 9400 1200
+F 0 "H1" H 9500 1246 50  0000 L CNN
+F 1 "MountingHole" H 9500 1155 50  0000 L CNN
+F 2 "MountingHole:MountingHole_2.5mm_Pad" H 9400 1200 50  0001 C CNN
+F 3 "~" H 9400 1200 50  0001 C CNN
+	1    9400 1200
+	1    0    0    -1
+$EndComp
+$Comp
+L Mechanical:MountingHole H2
+U 1 1 5DD37BCF
+P 9400 1400
+F 0 "H2" H 9500 1446 50  0000 L CNN
+F 1 "MountingHole" H 9500 1355 50  0000 L CNN
+F 2 "MountingHole:MountingHole_2.5mm_Pad" H 9400 1400 50  0001 C CNN
+F 3 "~" H 9400 1400 50  0001 C CNN
+	1    9400 1400
+	1    0    0    -1
+$EndComp
+$Comp
+L Mechanical:MountingHole H3
+U 1 1 5DD37E39
+P 9400 1600
+F 0 "H3" H 9500 1646 50  0000 L CNN
+F 1 "MountingHole" H 9500 1555 50  0000 L CNN
+F 2 "MountingHole:MountingHole_2.5mm_Pad" H 9400 1600 50  0001 C CNN
+F 3 "~" H 9400 1600 50  0001 C CNN
+	1    9400 1600
+	1    0    0    -1
+$EndComp
+$Comp
+L Mechanical:MountingHole H4
+U 1 1 5DD37F6A
+P 9400 1800
+F 0 "H4" H 9500 1846 50  0000 L CNN
+F 1 "MountingHole" H 9500 1755 50  0000 L CNN
+F 2 "MountingHole:MountingHole_2.5mm_Pad" H 9400 1800 50  0001 C CNN
+F 3 "~" H 9400 1800 50  0001 C CNN
+	1    9400 1800
+	1    0    0    -1
+$EndComp
 Wire Bus Line
 	2000 2500 3750 2500

Commit message: Correciones relizadas.
Parts:
- added FID1, FID2, FID3: Fiducial, Fiducial:Fiducial_0.5mm_Mask1mm, symbol Mechanical:Fiducial
Changed lines of the file:
@@
 Wire Bus Line
 	7950 4400 7950 6000
+$Comp
+L Mechanical:Fiducial FID1
+U 1 1 5DD8BA2C
+P 9400 2100
+F 0 "FID1" H 9485 2146 50  0000 L CNN
+F 1 "Fiducial" H 9485 2055 50  0000 L CNN
+F 2 "Fiducial:Fiducial_0.5mm_Mask1mm" H 9400 2100 50  0001 C CNN
+F 3 "~" H 9400 2100 50  0001 C CNN
+	1    9400 2100
+	1    0    0    -1
+$EndComp
+$Comp
+L Mechanical:Fiducial FID2
+U 1 1 5DD8BF4A
+P 9400 2300
+F 0 "FID2" H 9485 2346 50  0000 L CNN
+F 1 "Fiducial" H 9485 2255 50  0000 L CNN
+F 2 "Fiducial:Fiducial_0.5mm_Mask1mm" H 9400 2300 50  0001 C CNN
+F 3 "~" H 9400 2300 50  0001 C CNN
+	1    9400 2300
+	1    0    0    -1
+$EndComp
+$Comp
+L Mechanical:Fiducial FID3
+U 1 1 5DD8F9DD
+P 9400 2500
+F 0 "FID3" H 9485 2546 50  0000 L CNN
+F 1 "Fiducial" H 9485 2455 50  0000 L CNN
+F 2 "Fiducial:Fiducial_0.5mm_Mask1mm" H 9400 2500 50  0001 C CNN
+F 3 "~" H 9400 2500 50  0001 C CNN
+	1    9400 2500
+	1    0    0    -1
+$EndComp
 $EndSCHEMATC
